Commit message: rotate oliver tool 180

File: urdf/gp4_with_oliver_tool.xacro (robot description, xacro)
@@ -307,5 +307,5 @@
     </joint>
     <joint name="fts_tool" type="revolute">
-      <origin xyz="0 0 ${0.0505/2}" rpy="${pi/2} 0 ${-pi/2}" />
+      <origin xyz="0 0 ${0.0505/2}" rpy="${pi/2} 0 ${pi/2}" />
       <parent link="fts" />
       <child link="link_tool" />

Commit message: update tool

File: urdf/gp4_with_oliver_tool.xacro (robot description, xacro)
@@ -246,5 +246,5 @@
         <origin xyz="0 0 0" rpy="0 0 0"/>
         <geometry>
-          <mesh filename="file://$(find robot_digital_twin)/meshes/eoat/tool_with_hook.stl"/>
+          <mesh filename="file://$(find robot_digital_twin)/meshes/eoat/tool_hook_camera.stl"/>
         </geometry>
         <xacro:material_yaskawa_silver />
