Commit message: delete moveit package

File: urdf/dual_gp4.urdf (robot description, URDF)
Before this commit: robot dual_gp4, 30 links, 29 joints
Links:
- link base: mass 10.0 -> None; geometry 
- link left_arm_fts: geometry collision cylinder length=0.0505 radius=0.035; visual cylinder length=0.0505 radius=0.035
- link right_arm_fts: geometry collision cylinder length=0.0505 radius=0.035; visual cylinder length=0.0505 radius=0.035

File: urdf/dual_gp4.xacro (robot description, xacro)
@@ -9,24 +9,4 @@
     <!-- box shaped table as base for the 2 GP4 -->
     <link name="base">
-        <visual>
-            <origin xyz="0 0 -0.5" rpy="0 0 0" />
-            <geometry>z
-                <box size="2 2 1" />
-            </geometry>
-            <material name="White">
-                <color rgba="1.0 1.0 1.0 1.0" />
-            </material>
-        </visual>
-        <collision>
-            <origin xyz="0 0 -0.5" rpy="0 0 0" />
-            <geometry>
-                <box size="2 2 1" />
-            </geometry>
-        </collision>
-        <inertial>
-            <origin xyz="0.0 0.0 0.0" rpy="0.0 0.0 0.0"/>
-            <mass value="10.0"/>
-            <inertia ixx="0.001" ixy="0.0" ixz="0.001" iyy="0.0" iyz="0.0" izz="0.001"/>
-        </inertial>
     </link>
     <joint name="base_to_world" type="fixed">

Commit message: updated collision model

File: urdf/dual_gp4.urdf (robot description, URDF)
Before this commit: robot dual_gp4, 30 links, 29 joints
Links:
- removed link left_arm_link_camera
- removed link left_arm_link_camera_origin
- removed link left_arm_link_precam
- removed link right_arm_link_camera
- removed link right_arm_link_camera_origin
- removed link right_arm_link_precam
- link left_arm_base_link: geometry collision mesh filename=file:///home/philip/catkin_ws/src/robot_digital_twin/meshes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; visual mesh filename=file:///home/philip/catkin_ws/src/robot_digital_twin/meshes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
- link left_arm_link_1: geometry collision mesh filename=file:///home/philip/catkin_ws/src/robot_digital_twin/meshes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; visual mesh filename=file:///home/philip/catkin_ws/src/robot_digital_twin/meshes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
- link left_arm_link_2: geometry collision mesh filename=file:///home/philip/catkin_ws/src/robot_digital_twin/meshes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; visual mesh filename=file:///home/philip/catkin_ws/src/robot_digital_twin/meshes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
- link left_arm_link_3: geometry collision mesh filename=file:///home/philip/catkin_ws/src/robot_digital_twin/meshes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; visual mesh filename=file:///home/philip/catkin_ws/src/robot_digital_twin/meshes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
- link left_arm_link_4: geometry collision mesh filename=file:///home/philip/catkin_ws/src/robot_digital_twin/meshes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; visual mesh filename=file:///home/philip/catkin_ws/src/robot_digital_twin/meshes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
- link left_arm_link_5: geometry collision mesh filename=file:///home/philip/catkin_ws/src/robot_digital_twin/meshes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; visual mesh filename=file:///home/philip/catkin_ws/src/robot_digital_twin/meshes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
- link left_arm_link_6: geometry collision mesh filename=file:///home/philip/catkin_ws/src/robot_digital_twin/meshes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; visual mesh filename=file:///home/philip/catkin_ws/src/robot_digital_twin/meshes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
- link left_arm_link_tool: geometry collision mesh filename=file:///home/philip/catkin_ws/src/robot_digital_twin/meshes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; visual mesh filename=file:///home/philip/catkin_ws/src/robot_digital_twin/meshes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
- link right_arm_base_link: geometry collision mesh filename=file:///home/philip/catkin_ws/src/robot_digital_twin/meshes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; visual mesh filename=file:///home/philip/catkin_ws/src/robot_digital_twin/meshes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
- link right_arm_link_1: geometry collision mesh filename=file:///home/philip/catkin_ws/src/robot_digital_twin/meshes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; visual mesh filename=file:///home/philip/catkin_ws/src/robot_digital_twin/meshes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
- link right_arm_link_2: geometry collision mesh filename=file:///home/philip/catkin_ws/src/robot_digital_twin/meshes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; visual mesh filename=file:///home/philip/catkin_ws/src/robot_digital_twin/meshes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
- link right_arm_link_3: geometry collision mesh filename=file:///home/philip/catkin_ws/src/robot_digital_twin/meshes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; visual mesh filename=file:///home/philip/catkin_ws/src/robot_digital_twin/meshes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
- link right_arm_link_4: geometry collision mesh filename=file:///home/philip/catkin_ws/src/robot_digital_twin/meshes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; visual mesh filename=file:///home/philip/catkin_ws/src/robot_digital_twin/meshes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
- link right_arm_link_5: geometry collision mesh filename=file:///home/philip/catkin_ws/src/robot_digital_twin/meshes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; visual mesh filename=file:///home/philip/catkin_ws/src/robot_digital_twin/meshes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
- link right_arm_link_6: geometry collision mesh filename=file:///home/philip/catkin_ws/src/robot_digital_twin/meshes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; visual mesh filename=file:///home/philip/catkin_ws/src/robot_digital_twin/meshes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
- link right_arm_link_tool: geometry collision mesh filename=file:///home/philip/catkin_ws/src/robot_digital_twin/meshes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; visual mesh filename=file:///home/philip/catkin_ws/src/robot_digital_twin/meshes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
Joints:
- removed joint left_arm_camera_imgplane
- removed joint left_arm_precam_camera
- removed joint left_arm_tool_precam
- removed joint right_arm_camera_imgplane
- removed joint right_arm_precam_camera
- removed joint right_arm_tool_precam
- joint right_arm_to_base: origin xyz=0.7951 0 0.9246 rpy=0 0 3.141592653589793 -> xyz=0.8782 -0.0115 0.9246 rpy=0 0 3.15119196

File: urdf/single_gp4.xacro (robot description, xacro)
@@ -75,5 +75,5 @@
       <collision>
         <geometry>
-          <mesh filename="file://$(find robot_digital_twin)/meshes/gp4/link_1.stl"/>
+          <mesh filename="file://$(find robot_digital_twin)/meshes/gp4/link_1_scaled.stl"/>
         </geometry>
       </collision>
@@ -102,5 +102,5 @@
       <collision>
         <geometry>
-          <mesh filename="file://$(find robot_digital_twin)/meshes/gp4/link_2.stl"/>
+          <mesh filename="file://$(find robot_digital_twin)/meshes/gp4/link_2_scaled.stl"/>
         </geometry>
       </collision>
@@ -129,5 +129,5 @@
       <collision>
         <geometry>
-          <mesh filename="file://$(find robot_digital_twin)/meshes/gp4/link_3.stl"/>
+          <mesh filename="file://$(find robot_digital_twin)/meshes/gp4/link_3_scaled.stl"/>
         </geometry>
       </collision>
@@ -156,5 +156,5 @@
       <collision>
         <geometry>
-          <mesh filename="file://$(find robot_digital_twin)/meshes/gp4/link_4.stl"/>
+          <mesh filename="file://$(find robot_digital_twin)/meshes/gp4/link_4_scaled.stl"/>
         </geometry>
       </collision>
@@ -183,5 +183,5 @@
       <collision>
         <geometry>
-          <mesh filename="file://$(find robot_digital_twin)/meshes/gp4/link_5.stl"/>
+          <mesh filename="file://$(find robot_digital_twin)/meshes/gp4/link_5_scaled.stl"/>
         </geometry>
       </collision>
@@ -210,5 +210,5 @@
       <collision>
         <geometry>
-          <mesh filename="file://$(find robot_digital_twin)/meshes/gp4/link_6.stl"/>
+          <mesh filename="file://$(find robot_digital_twin)/meshes/gp4/link_6_scaled.stl"/>
         </geometry>
       </collision>
@@ -218,5 +218,5 @@
         <origin xyz="0 0 0" rpy=" 0 0 0"/>
         <geometry>
-          <cylinder length="0.0505" radius="0.035"/>
+          <cylinder length="0.0505" radius="0.03675"/>
         </geometry>
       </collision>
@@ -262,59 +262,4 @@
         <xacro:material_yaskawa_silver />
       </visual>
-    </link>
-    <link name="${arm_id}_link_precam">
-      <inertial>
-        <mass value="1e-5" />
-        <origin xyz="0 0 0" rpy="0 0 0"/>
-        <inertia ixx="1e-6" ixy="0" ixz="0" iyy="1e-6" iyz="0" izz="1e-6" />
-      </inertial>
-    </link>
-    <link name="${arm_id}_link_camera">
-    <inertial>
-      <origin
-        xyz="0 0 0"
-        rpy="0 0 0" />
-      <mass
-        value="0.10811" />
-      <inertia
-        ixx="9.0129E-05"
-        ixy="-1.0891E-08"
-        ixz="9.1598E-09"
-        iyy="9.2026E-05"
-        iyz="-2.749E-07"
-        izz="0.00017818" />
-    </inertial>
-      <visual>
-        <origin xyz="0 0 0" rpy="0 0 0"/>
-        <geometry>
-          <mesh filename="file://$(find robot_digital_twin)/meshes/eoat/tool_camera.stl"/>
-        </geometry>
-        <xacro:material_fanuc_black />
-      </visual>
-      <collision>
-        <origin xyz="0 0 0" rpy="0 0 0"/>
-        <geometry>
-          <mesh filename="file://$(find robot_digital_twin)/meshes/eoat/tool_camera.stl"/>
-        </geometry>
-      </collision>
-    </link>
-    <link name="${arm_id}_link_camera_origin">
-    <collision>
-      <origin xyz="0 0 0" rpy="0 0 0"/>
-      <geometry>
-        <box size="0.0001 0.0001 0.0001"/>
-      </geometry>
-    </collision>
-    <visual>
-      <origin xyz="0 0 0" rpy="0 0 0"/>
-      <geometry>
-        <box size="0.0001 0.01 0.01"/>
-      </geometry>
-    </visual>
-      <inertial>
-        <mass value="1e-5" />
-        <origin xyz="0 0 0" rpy="0 0 0"/>
-        <inertia ixx="1e-6" ixy="0" ixz="0" iyy="1e-6" iyz="0" izz="1e-6" />
-      </inertial>
     </link>
     <!-- joints: main serial chain -->
@@ -379,19 +324,4 @@
       <axis xyz="0 0 1" />
       <limit velocity="0" effort="0" lower="0" upper="0" />
-    </joint>
-    <joint name="${arm_id}_tool_precam" type="fixed">
-      <origin xyz="0 -0.062194148 -0.005909903" rpy="${pi/2} -${pi/2}  0" />
-      <parent link="${arm_id}_link_tool" />
-      <child link="${arm_id}_link_precam" />
-    </joint>
-    <joint name="${arm_id}_precam_camera" type="fixed">
-      <origin xyz="0 0 0" rpy="0 ${pi*45/180} 0" />
-      <parent link="${arm_id}_link_precam" />
-      <child link="${arm_id}_link_camera" />
-    </joint>
-    <joint name="${arm_id}_camera_imgplane" type="fixed">
-      <origin xyz="0.013 0.0 0.0305" rpy="0 0 0" />
-      <parent link="${arm_id}_link_camera" />
-      <child link="${arm_id}_link_camera_origin" />
     </joint>
   </xacro:macro>
@@ -434,40 +364,4 @@
         </plugin>
     </gazebo>
-    <gazebo reference="link_camera_origin">
-    <sensor name="$depth_camera" type="depth">
-      <update_rate>30</update_rate>
-      <camera>
-        <horizontal_fov>1.22173</horizontal_fov> <!-- 70deg -->
-        <image>
-          <width>1920</width>
-          <height>1080</height>
-          <format>R8G8B8</format>
-        </image>
-        <clip>
-          <near>0.005</near>
-          <far>2</far>
-        </clip>
-      </camera>
-      <plugin name="$depth_camera_controller" filename="libgazebo_ros_openni_kinect.so">
-        <baseline>0.2</baseline>
-        <alwaysOn>true</alwaysOn>
-        <updateRate>0</updateRate>
-        <cameraName>${arm_id}_wrist_camera</cameraName>
-        <frameName>${arm_id}_depth_camera_link</frameName>
-        <pointCloudCutoff>0.005</pointCloudCutoff>
-        <pointCloudCutoffMax>2.0</pointCloudCutoffMax>
-        <distortionK1>0</distortionK1>
-        <distortionK2>0</distortionK2>
-        <distortionK3>0</distortionK3>
-        <distortionT1>0</distortionT1>
-        <distortionT2>0</distortionT2>
-        <CxPrime>0</CxPrime>
-        <Cx>0</Cx>
-        <Cy>0</Cy>
-        <focalLength>0</focalLength>
-        <hackBaseline>0</hackBaseline>
-      </plugin>
-    </sensor>
-  </gazebo>
     <gazebo reference="${arm_id}_base">
       <material>Gazebo/Blue</material>
@@ -510,8 +404,4 @@
       <visual> <transparency> 0 </transparency> </visual>
     </gazebo>
-    <gazebo reference="${arm_id}_link_camera_origin">
-      <material>Gazebo/Black</material>
-      <visual> <transparency> 0 </transparency> </visual>
-    </gazebo>
   </xacro:macro>
 </robot>

Commit message: make calibration between urdf and txt consistent, still need to do more test

File: urdf/dual_gp4.urdf (robot description, URDF)
Before this commit: robot dual_gp4, 24 links, 23 joints
Links:
- link left_arm_fts: geometry collision cylinder length=0.0505 radius=0.058; visual cylinder length=0.0505 radius=0.0472
- link right_arm_fts: geometry collision cylinder length=0.0505 radius=0.058; visual cylinder length=0.0505 radius=0.0472
Joints:
- joint right_arm_to_base: origin xyz=0.8782 -0.0115 0.9246 rpy=0 0 3.15119196 -> xyz=0.87871678 -0.01878527 0.92578 rpy=0 0 3.1412068136520546

File: urdf/dual_gp4.urdf.xacro (robot description, xacro)
@@ -19,5 +19,5 @@
     <!-- left arm gazebo -->
     <!-- right arm -->
-    <xacro:Yaskawa_gp4 arm_id="$(arg arm_id_2)" connected_to="base" xyz="0.87871678 -0.01878527 0.92578" rpy="0 0 3.1412068136520546" />
+    <xacro:Yaskawa_gp4 arm_id="$(arg arm_id_2)" connected_to="base" xyz="0.87739561 -0.02770527 0.92578" rpy="0 0 3.10048065" />
     <!-- right arm gazebo-->
     <xacro:gp4_gazebo arm_id="$(arg arm_id_2)" />
