Commit message: update

File: urdf/lego_1x1.xacro (robot description, xacro)
@@ -73,4 +73,7 @@
      <material>Gazebo/Grey</material>
     </xacro:if>
+    <xacro:if value="${color == 'Purple'}">
+     <material>Gazebo/Purple</material>
+    </xacro:if>
     <visual> <transparency> 0 </transparency> </visual>
   </gazebo>

File: urdf/lego_1x2.xacro (robot description, xacro)
@@ -73,4 +73,7 @@
      <material>Gazebo/Grey</material>
     </xacro:if>
+    <xacro:if value="${color == 'Purple'}">
+     <material>Gazebo/Purple</material>
+    </xacro:if>
     <visual> <transparency> 0 </transparency> </visual>
   </gazebo>

File: urdf/lego_1x4.xacro (robot description, xacro)
@@ -73,4 +73,7 @@
      <material>Gazebo/Grey</material>
     </xacro:if>
+    <xacro:if value="${color == 'Purple'}">
+     <material>Gazebo/Purple</material>
+    </xacro:if>
     <visual> <transparency> 0 </transparency> </visual>
   </gazebo>

File: urdf/lego_1x6.xacro (robot description, xacro)
@@ -73,4 +73,7 @@
      <material>Gazebo/Grey</material>
     </xacro:if>
+    <xacro:if value="${color == 'Purple'}">
+     <material>Gazebo/Purple</material>
+    </xacro:if>
     <visual> <transparency> 0 </transparency> </visual>
   </gazebo>

File: urdf/lego_1x8.xacro (robot description, xacro)
@@ -73,4 +73,7 @@
      <material>Gazebo/Grey</material>
     </xacro:if>
+    <xacro:if value="${color == 'Purple'}">
+     <material>Gazebo/Purple</material>
+    </xacro:if>
     <visual> <transparency> 0 </transparency> </visual>
   </gazebo>

File: urdf/lego_2x2.xacro (robot description, xacro)
@@ -73,4 +73,7 @@
      <material>Gazebo/Grey</material>
     </xacro:if>
+    <xacro:if value="${color == 'Purple'}">
+     <material>Gazebo/Purple</material>
+    </xacro:if>
     <visual> <transparency> 0 </transparency> </visual>
   </gazebo>

File: urdf/lego_2x4.xacro (robot description, xacro)
@@ -73,4 +73,7 @@
      <material>Gazebo/Grey</material>
     </xacro:if>
+    <xacro:if value="${color == 'Purple'}">
+     <material>Gazebo/Purple</material>
+    </xacro:if>
     <visual> <transparency> 0 </transparency> </visual>
   </gazebo>

File: urdf/lego_2x6.xacro (robot description, xacro)
@@ -73,4 +73,7 @@
      <material>Gazebo/Grey</material>
     </xacro:if>
+    <xacro:if value="${color == 'Purple'}">
+     <material>Gazebo/Purple</material>
+    </xacro:if>
     <visual> <transparency> 0 </transparency> </visual>
   </gazebo>

File: urdf/lego_2x8.xacro (robot description, xacro)
@@ -73,4 +73,7 @@
      <material>Gazebo/Grey</material>
     </xacro:if>
+    <xacro:if value="${color == 'Purple'}">
+     <material>Gazebo/Purple</material>
+    </xacro:if>
     <visual> <transparency> 0 </transparency> </visual>
   </gazebo>

File: urdf/lego_baseplate.xacro (robot description, xacro)
@@ -73,4 +73,7 @@
      <material>Gazebo/Grey</material>
     </xacro:if>
+    <xacro:if value="${color == 'Purple'}">
+     <material>Gazebo/Purple</material>
+    </xacro:if>
     <visual> <transparency> 0 </transparency> </visual>
   </gazebo>

File: urdf/lego_baseplate32.xacro (robot description, xacro)
@@ -73,4 +73,7 @@
      <material>Gazebo/Grey</material>
     </xacro:if>
+    <xacro:if value="${color == 'Purple'}">
+     <material>Gazebo/Purple</material>
+    </xacro:if>
     <visual> <transparency> 0 </transparency> </visual>
   </gazebo>

File: urdf/lego_baseplate48.xacro (robot description, xacro)
@@ -73,4 +73,7 @@
      <material>Gazebo/Grey</material>
     </xacro:if>
+    <xacro:if value="${color == 'Purple'}">
+     <material>Gazebo/Purple</material>
+    </xacro:if>
     <visual> <transparency> 0 </transparency> </visual>
   </gazebo>
