Commit message: update tool

File: urdf/fanuc_arm.xacro (robot description, xacro)
@@ -259,14 +259,21 @@
         <origin xyz="0 0 0" rpy="0 0 0"/>
         <geometry>
+          <mesh filename="file://$(find robot_digital_twin)/meshes/eoat/tool_base_tilt.stl"/>
+        </geometry>
+        <xacro:material_fanuc_black />
+      </visual>
+      <!-- <collision>
+        <origin xyz="0 0 0" rpy="0 0 0"/>
+        <geometry>
           <mesh filename="file://$(find robot_digital_twin)/meshes/eoat/tool_base.stl"/>
         </geometry>
-        <xacro:material_fanuc_black />
-      </visual>
-      <!-- <collision>
-        <origin xyz="0 0 0" rpy="0 0 0"/>
-        <geometry>
-          <mesh filename="file://$(find robot_digital_twin)/meshes/eoat/tool_base.stl"/>
-        </geometry>
       </collision> -->
+    </link>
+    <link name="link_precam">
+      <inertial>
+        <mass value="1e-5" />
+        <origin xyz="0 0 0" rpy="0 0 0"/>
+        <inertia ixx="1e-6" ixy="0" ixz="0" iyy="1e-6" iyz="0" izz="1e-6" />
+      </inertial>
     </link>
     <link name="link_camera">
@@ -373,7 +380,12 @@
       <limit velocity="0" effort="0" lower="0" upper="0" />
     </joint>
-    <joint name="tool_camera" type="fixed">
-      <origin xyz="0 -0.04625 0.028" rpy="${-pi/2.0} ${-pi/2.0} ${pi}" />
+    <joint name="tool_precam" type="fixed">
+      <origin xyz="0 -0.062194148 -0.005909903" rpy="${pi/2} -${pi/2}  0" />
       <parent link="link_tool" />
+      <child link="link_precam" />
+    </joint>
+    <joint name="precam_camera" type="fixed">
+      <origin xyz="0 0 0" rpy="0 ${pi*45/180} 0" />
+      <parent link="link_precam" />
       <child link="link_camera" />
     </joint>

Commit message: update tool height

File: urdf/fanuc_arm.xacro (robot description, xacro)
@@ -259,5 +259,5 @@
         <origin xyz="0 0 0" rpy="0 0 0"/>
         <geometry>
-          <mesh filename="file://$(find robot_digital_twin)/meshes/eoat/tool_base_tilt.stl"/>
+          <mesh filename="file://$(find robot_digital_twin)/meshes/eoat/tool_base.stl"/>
         </geometry>
         <xacro:material_fanuc_black />

File: urdf/gp4.xacro (robot description, xacro)
@@ -246,5 +246,5 @@
         <origin xyz="0 0 0" rpy="0 0 0"/>
         <geometry>
-          <mesh filename="file://$(find robot_digital_twin)/meshes/eoat/tool_base_tilt.stl"/>
+          <mesh filename="file://$(find robot_digital_twin)/meshes/eoat/tool_base.stl"/>
         </geometry>
         <xacro:material_yaskawa_silver />

File: urdf/single_gp4.xacro (robot description, xacro)
@@ -252,5 +252,5 @@
       <origin xyz="0 0 0" rpy="0 0 0"/>
       <geometry>
-        <mesh filename="file://$(find robot_digital_twin)/meshes/eoat/tool_base_tilt.stl"/>
+        <mesh filename="file://$(find robot_digital_twin)/meshes/eoat/tool_base.stl"/>
       </geometry>
     </collision>
@@ -258,5 +258,5 @@
         <origin xyz="0 0 0" rpy="0 0 0"/>
         <geometry>
-          <mesh filename="file://$(find robot_digital_twin)/meshes/eoat/tool_base_tilt.stl"/>
+          <mesh filename="file://$(find robot_digital_twin)/meshes/eoat/tool_base.stl"/>
         </geometry>
         <xacro:material_yaskawa_silver />

Commit message: add plates models

File: urdf/fanuc_arm.xacro (robot description, xacro)
@@ -219,5 +219,5 @@
         <geometry>
           <mesh filename="file://$(find robot_digital_twin)/meshes/lrmate200id_7L/link_6.stl"/>
-        </geometry>
+        </geometry>fanuc_arm
       </collision>
     </link>
