Commit message: fix g1 color in gazebo

File: urdf/g1_single_arm.urdf (robot description, URDF)
Before this commit: robot g1_single_arm, 10 links, 9 joints
Links:
- link virtual_right_wrist_link: geometry 

Commit message: add g1 fixed base link

File: urdf/g1_single_arm.urdf (robot description, URDF)
Before this commit: robot g1_single_arm, 10 links, 9 joints
Links:
- added link waist_roll_link, mass 0.047; visual mesh filename=meshes/waist_roll_link.STL
- added link waist_yaw_link, mass 0.244; visual mesh filename=meshes/waist_yaw_link.STL
Joints:
- added joint waist_roll_joint: type fixed, parent waist_yaw_link, child waist_roll_link, origin xyz=-0.0039635 0 0.035 rpy=0 0 0, axis 1 0 0, limit lower=-0.52 upper=0.52 effort=50 velocity=37
- added joint waist_yaw_joint: type fixed, parent world, child waist_yaw_link, origin xyz=0 0 0 rpy=0 0 0
- joint waist_pitch_joint: parent world -> waist_roll_link

Commit message: add g1 wrist yaw

File: urdf/g1_single_arm.urdf (robot description, URDF)
Before this commit: robot g1_single_arm, 12 links, 11 joints
Links:
- added link pelvis, mass 3.813; visual mesh filename=meshes/pelvis.STL
Joints:
- added joint pelvis_joint: type fixed, parent world, child pelvis, origin xyz=0 0 0 rpy=0 0 0
- joint right_wrist_roll_joint: axis 1 0 0 -> (none); limit lower=-1.972222054 upper=1.972222054 effort=25 velocity=37 -> (none); type revolute -> fixed
- joint waist_yaw_joint: axis (none) -> 0 0 1; limit (none) -> lower=-2.618 upper=2.618 effort=88 velocity=32; parent world -> pelvis; type fixed -> revolute

Commit message: fix mesh path

File: urdf/g1_single_arm.urdf (robot description, URDF)
Before this commit: robot g1_single_arm, 13 links, 12 joints
Links:
- link pelvis: geometry visual mesh filename=package://robot_digital_twin/meshes/g1/pelvis.STL
- link waist_roll_link: geometry visual mesh filename=package://robot_digital_twin/meshes/g1/waist_roll_link.STL
- link waist_yaw_link: geometry visual mesh filename=package://robot_digital_twin/meshes/g1/waist_yaw_link.STL

Commit message: custom joint range

File: urdf/g1_single_arm.urdf (robot description, URDF)
Before this commit: robot g1_single_arm, 13 links, 12 joints
Joints:
- joint right_shoulder_roll_joint: limit lower=-2.2515 upper=1.5882 effort=25 velocity=37 -> lower=-2.2515 upper=0.3 effort=25 velocity=37
- joint waist_pitch_joint: limit lower=-0.52 upper=0.52 effort=50 velocity=37 -> lower=0.0 upper=0.52 effort=50 velocity=37
- joint waist_yaw_joint: limit lower=-2.618 upper=2.618 effort=88 velocity=32 -> lower=-1.0 upper=1.0 effort=88 velocity=32
