Commit message: block assembly

File: urdf/block.xacro (robot description, xacro)
@@ -3,7 +3,7 @@
   name="block" xmlns:xacro="http://ros.org/wiki/xacro">
   <xacro:macro name="block">
-  <xacro:arg name="fruit_color" default="Red" />
+  <xacro:arg name="color" default="Red" />
   <xacro:property name="scale" value="1"/>
-  <xacro:property name="color" value="$(arg fruit_color)"/>
+  <xacro:property name="color" value="$(arg color)"/>
   <link
     name="block">
@@ -49,8 +49,8 @@
       </gazebo>
     </collision>
-    <gravity>true</gravity>
+    <gravity>1</gravity>
   </link>
   <gazebo reference="block">
-  <kinematic>false</kinematic>
+  <kinematic>0</kinematic>
   <xacro:if value="${color == 'Orange'}">
      <material>Gazebo/Orange</material>
