Commit message: update robot model and calibration

File: urdf/dual_gp4.urdf.xacro (robot description, xacro)
@@ -19,5 +19,5 @@
     <!-- left arm gazebo -->
     <!-- right arm -->
-    <xacro:Yaskawa_gp4 arm_id="$(arg arm_id_2)" connected_to="base" xyz="0.88047659 -0.01305078 0.9246" rpy="0 0 3.13422265" />
+    <xacro:Yaskawa_gp4 arm_id="$(arg arm_id_2)" connected_to="base" xyz="0.88061454 -0.01327456 0.9246" rpy="0 0 3.136692653589793" />
     <!-- right arm gazebo-->
     <xacro:gp4_gazebo arm_id="$(arg arm_id_2)" />

File: urdf/single_gp4.xacro (robot description, xacro)
@@ -259,5 +259,5 @@
         <origin xyz="0 0 0" rpy="0 0 0"/>
         <geometry>
-          <mesh filename="file://$(find robot_digital_twin)/meshes/eoat/D405_mount.stl"/>
+          <mesh filename="file://$(find robot_digital_twin)/meshes/eoat/D405_mount_inflated.stl"/>
         </geometry>
       </collision>
@@ -295,5 +295,5 @@
         <origin xyz="0 0 0" rpy="0 0 0"/>
         <geometry>
-          <mesh filename="file://$(find robot_digital_twin)/meshes/eoat/D405.stl"/>
+          <mesh filename="file://$(find robot_digital_twin)/meshes/eoat/D405_inflated.stl"/>
         </geometry>
       </collision>
