Commit message: ready for test 12_11

File: urdf/fanuc_3f_gripper.xacro (robot description, xacro)
@@ -727,5 +727,5 @@
   <xacro:fanuc_lrmate200id7l>
   </xacro:fanuc_lrmate200id7l>
-  <xacro:macro name="transmission_block" params="joint_name">
+  <xacro:macro name="position_transmission_block" params="joint_name">
     <transmission name = "trans_${joint_name}">
       <type>transmission_interface/SimpleTransmission</type>
@@ -739,22 +739,34 @@
     </transmission>
   </xacro:macro>
-  <xacro:transmission_block joint_name = "joint_1"/>
-  <xacro:transmission_block joint_name = "joint_2"/>
-  <xacro:transmission_block joint_name = "joint_3"/>
-  <xacro:transmission_block joint_name = "joint_4"/>
-  <xacro:transmission_block joint_name = "joint_5"/>
-  <xacro:transmission_block joint_name = "joint_6"/>
-  <xacro:transmission_block joint_name = "finger_A_joint_0"/>
-  <xacro:transmission_block joint_name = "finger_A_joint_1"/>
-  <xacro:transmission_block joint_name = "finger_A_joint_2"/>
-  <xacro:transmission_block joint_name = "finger_A_joint_3"/>
-  <xacro:transmission_block joint_name = "finger_B_joint_0"/>
-  <xacro:transmission_block joint_name = "finger_B_joint_1"/>
-  <xacro:transmission_block joint_name = "finger_B_joint_2"/>
-  <xacro:transmission_block joint_name = "finger_B_joint_3"/>
-  <xacro:transmission_block joint_name = "finger_C_joint_0"/>
-  <xacro:transmission_block joint_name = "finger_C_joint_1"/>
-  <xacro:transmission_block joint_name = "finger_C_joint_2"/>
-  <xacro:transmission_block joint_name = "finger_C_joint_3"/>
+  <xacro:macro name="effort_transmission_block" params="joint_name">
+    <transmission name = "trans_${joint_name}">
+      <type>transmission_interface/SimpleTransmission</type>
+      <joint name = "${joint_name}">
+        <hardwareInterface>hardware_interface/EffortJointInterface</hardwareInterface>
+      </joint>
+      <actuator name = "${joint_name}_motor">
+        <hardwareInterface>hardware_interface/EffortJointInterface</hardwareInterface>
+        <mechanicalReduction>1</mechanicalReduction>
+      </actuator>
+    </transmission>
+  </xacro:macro>
+  <xacro:position_transmission_block joint_name = "joint_1"/>
+  <xacro:position_transmission_block joint_name = "joint_2"/>
+  <xacro:position_transmission_block joint_name = "joint_3"/>
+  <xacro:position_transmission_block joint_name = "joint_4"/>
+  <xacro:position_transmission_block joint_name = "joint_5"/>
+  <xacro:position_transmission_block joint_name = "joint_6"/>
+  <xacro:position_transmission_block joint_name = "finger_A_joint_0"/>
+  <xacro:position_transmission_block joint_name = "finger_A_joint_1"/>
+  <xacro:position_transmission_block joint_name = "finger_A_joint_2"/>
+  <xacro:position_transmission_block joint_name = "finger_A_joint_3"/>
+  <xacro:position_transmission_block joint_name = "finger_B_joint_0"/>
+  <xacro:position_transmission_block joint_name = "finger_B_joint_1"/>
+  <xacro:position_transmission_block joint_name = "finger_B_joint_2"/>
+  <xacro:position_transmission_block joint_name = "finger_B_joint_3"/>
+  <xacro:position_transmission_block joint_name = "finger_C_joint_0"/>
+  <xacro:position_transmission_block joint_name = "finger_C_joint_1"/>
+  <xacro:position_transmission_block joint_name = "finger_C_joint_2"/>
+  <xacro:position_transmission_block joint_name = "finger_C_joint_3"/>
   <gazebo>
     <plugin name="gazebo_ros_control" filename="libgazebo_ros_control.so">
@@ -769,21 +781,21 @@
            <arm_name>fanuc_arm_/fanuc_gazebo/</arm_name>
            <palm_link> link_6  </palm_link>
-           <gripper_link> finger_A_link_0 </gripper_link>
+           <!-- <gripper_link> finger_A_link_0 </gripper_link>
            <gripper_link> finger_A_link_1 </gripper_link>
-           <gripper_link> finger_A_link_2 </gripper_link>
+           <gripper_link> finger_A_link_2 </gripper_link> -->
            <gripper_link> finger_A_link_3 </gripper_link>
-           <gripper_link> finger_B_link_0 </gripper_link>
+           <!-- <gripper_link> finger_B_link_0 </gripper_link>
            <gripper_link> finger_B_link_1 </gripper_link>
-           <gripper_link> finger_B_link_2 </gripper_link>
+           <gripper_link> finger_B_link_2 </gripper_link> -->
            <gripper_link> finger_B_link_3 </gripper_link>
-           <gripper_link> finger_C_link_0 </gripper_link>
+           <!-- <gripper_link> finger_C_link_0 </gripper_link>
            <gripper_link> finger_C_link_1 </gripper_link>
-           <gripper_link> finger_C_link_2 </gripper_link>
+           <gripper_link> finger_C_link_2 </gripper_link> -->
            <gripper_link> finger_C_link_3 </gripper_link>
         </arm>
-       <forces_angle_tolerance>90</forces_angle_tolerance>
+       <forces_angle_tolerance>180</forces_angle_tolerance>
        <update_rate>20</update_rate>
-       <grip_count_threshold>2</grip_count_threshold>
-       <max_grip_count>50</max_grip_count>
+       <grip_count_threshold>1</grip_count_threshold>
+       <max_grip_count>100</max_grip_count>
        <release_tolerance>0.005</release_tolerance>
        <disable_collisions_on_attach>true</disable_collisions_on_attach>

File: urdf/g1_29dof_fixed.urdf (robot description, URDF)
Before this commit: robot g1_29dof, 42 links, 41 joints
Joints:
- joint left_elbow_joint: type revolute -> fixed
- joint left_shoulder_pitch_joint: type revolute -> fixed
- joint left_shoulder_roll_joint: type revolute -> fixed
- joint left_shoulder_yaw_joint: type revolute -> fixed
- joint left_wrist_pitch_joint: type revolute -> fixed
- joint left_wrist_roll_joint: type revolute -> fixed
- joint left_wrist_yaw_joint: type revolute -> fixed
- joint right_elbow_joint: type revolute -> fixed
- joint right_shoulder_pitch_joint: type revolute -> fixed
- joint right_shoulder_roll_joint: type revolute -> fixed
- joint right_shoulder_yaw_joint: type revolute -> fixed
- joint right_wrist_pitch_joint: type revolute -> fixed
- joint right_wrist_roll_joint: type revolute -> fixed
- joint right_wrist_yaw_joint: type revolute -> fixed
- joint waist_pitch_joint: type revolute -> fixed
- joint waist_roll_joint: type revolute -> fixed
- joint waist_yaw_joint: type revolute -> fixed
