Commit message: update gp4 collision model

File: urdf/single_gp4.xacro (robot description, xacro)
@@ -218,5 +218,5 @@
         <origin xyz="0 0 0" rpy=" 0 0 0"/>
         <geometry>
-          <cylinder length="0.0505" radius="0.03675"/>
+          <cylinder length="0.0505" radius="0.058"/>
         </geometry>
       </collision>
@@ -224,5 +224,5 @@
         <origin xyz="0 0 0" rpy="0 0 0"/>
         <geometry>
-          <cylinder length="0.0505" radius="0.035"/>
+          <cylinder length="0.0505" radius="0.0472"/>
         </geometry>
         <xacro:material_yaskawa_silver />

Commit message: update the single gp4 xacro used in moveit package

File: urdf/single_gp4.xacro (robot description, xacro)
@@ -234,5 +234,5 @@
       </inertial>
     </link>
-    <link name="${arm_id}_link_tool">
+    <link name="${arm_id}_link_mountplate">
     <inertial>
       <origin
@@ -249,8 +249,86 @@
         izz="0.00017818" />
     </inertial>
+      <visual>
+        <origin xyz="0 0 0" rpy="0 0 0"/>
+        <geometry>
+          <mesh filename="file://$(find robot_digital_twin)/meshes/eoat/D405_mount.stl"/>
+        </geometry>
+        <xacro:material_yaskawa_silver />
+      </visual>
+      <collision>
+        <origin xyz="0 0 0" rpy="0 0 0"/>
+        <geometry>
+          <mesh filename="file://$(find robot_digital_twin)/meshes/eoat/D405_mount.stl"/>
+        </geometry>
+      </collision>
+    </link>
+    <link name="${arm_id}_link_precam">
+      <inertial>
+        <mass value="1e-5" />
+        <origin xyz="0 0 0" rpy="0 0 0"/>
+        <inertia ixx="1e-6" ixy="0" ixz="0" iyy="1e-6" iyz="0" izz="1e-6" />
+      </inertial>
+    </link>
+    <link name="${arm_id}_link_camera">
+    <inertial>
+      <origin
+        xyz="0 0 0"
+        rpy="0 0 0" />
+      <mass
+        value="0.10811" />
+      <inertia
+        ixx="9.0129E-05"
+        ixy="-1.0891E-08"
+        ixz="9.1598E-09"
+        iyy="9.2026E-05"
+        iyz="-2.749E-07"
+        izz="0.00017818" />
+    </inertial>
+      <visual>
+        <origin xyz="0 0 0" rpy="0 0 0"/>
+        <geometry>
+          <mesh filename="file://$(find robot_digital_twin)/meshes/eoat/D405.stl"/>
+        </geometry>
+        <xacro:material_fanuc_black />
+      </visual>
+      <collision>
+        <origin xyz="0 0 0" rpy="0 0 0"/>
+        <geometry>
+          <mesh filename="file://$(find robot_digital_twin)/meshes/eoat/D405.stl"/>
+        </geometry>
+      </collision>
+    </link>
+    <link name="${arm_id}_link_camera_origin">
+    <visual>
+      <origin xyz="0 0 0" rpy="0 0 0"/>
+      <geometry>
+        <box size="0.0001 0.002 0.001"/>
+      </geometry>
+    </visual>
+      <inertial>
+        <mass value="1e-5" />
+        <origin xyz="0 0 0" rpy="0 0 0"/>
+        <inertia ixx="1e-6" ixy="0" ixz="0" iyy="1e-6" iyz="0" izz="1e-6" />
+      </inertial>
+    </link>
+    <link name="${arm_id}_link_tool">
+    <inertial>
+      <origin
+        xyz="0 0 0"
+        rpy="0 0 0" />
+      <mass
+        value="0.10811" />
+      <inertia
+        ixx="9.0129E-05"
+        ixy="-1.0891E-08"
+        ixz="9.1598E-09"
+        iyy="9.2026E-05"
+        iyz="-2.749E-07"
+        izz="0.00017818" />
+    </inertial>
     <collision>
       <origin xyz="0 0 0" rpy="0 0 0"/>
       <geometry>
-        <mesh filename="file://$(find robot_digital_twin)/meshes/eoat/tool_base.stl"/>
+        <mesh filename="file://$(find robot_digital_twin)/meshes/eoat/tool.stl"/>
       </geometry>
     </collision>
@@ -258,5 +336,5 @@
         <origin xyz="0 0 0" rpy="0 0 0"/>
         <geometry>
-          <mesh filename="file://$(find robot_digital_twin)/meshes/eoat/tool_base.stl"/>
+          <mesh filename="file://$(find robot_digital_twin)/meshes/eoat/tool.stl"/>
         </geometry>
         <xacro:material_yaskawa_silver />
@@ -318,6 +396,26 @@
       <child link="${arm_id}_fts" />
     </joint>
+    <joint name="${arm_id}_fts_plate" type="fixed">
+      <origin xyz="0 0 ${0.0505/2+0.00001}" rpy="${pi/2.0} 0 0" />
+      <parent link="${arm_id}_fts" />
+      <child link="${arm_id}_link_mountplate" />
+    </joint>
+    <joint name="${arm_id}_plate_precam" type="fixed">
+      <origin xyz="0 0 0" rpy="-${pi/2.0} 0  0" />
+      <parent link="${arm_id}_link_mountplate" />
+      <child link="${arm_id}_link_precam" />
+    </joint>
+    <joint name="${arm_id}_precam_camera" type="fixed">
+      <origin xyz="0 0.053512 ${0.00254+0.023+0.00001}" rpy="0  0  0" />
+      <parent link="${arm_id}_link_precam" />
+      <child link="${arm_id}_link_camera" />
+    </joint>
+    <joint name="${arm_id}_camera_imgplane" type="fixed">
+      <origin xyz="0.009 0 0" rpy="0 ${pi/2 + pi} -${pi/2}" />
+      <parent link="${arm_id}_link_camera" />
+      <child link="${arm_id}_link_camera_origin" />
+    </joint>
     <joint name="${arm_id}_fts_tool" type="revolute">
-      <origin xyz="0 0 ${0.0505/2}" rpy="0 0 ${pi}" />
+      <origin xyz="0 0 ${0.0505/2 + 0.00254}" rpy="0 0 ${pi}" />
       <parent link="${arm_id}_fts" />
       <child link="${arm_id}_link_tool" />

Commit message: update gp4 joint angle limits to revolute

File: urdf/single_gp4.xacro (robot description, xacro)
@@ -342,5 +342,5 @@
     </link>
     <!-- joints: main serial chain -->
-    <joint name="${arm_id}_joint_1" type="continuous">
+    <joint name="${arm_id}_joint_1" type="revolute">
       <parent link="${arm_id}_base_link"/>
       <child link="${arm_id}_link_1"/>
@@ -348,40 +348,40 @@
       <axis xyz="0 0 1" />
       <!-- <limit lower="${radians(-170)}" upper="${radians(170)}" effort="220.5" velocity="${radians(465)}"/> -->
-      <!-- <limit effort="0" lower="${radians(-170)}" upper="${radians(170)}" velocity="${radians(370)}" /> -->
-    </joint>
-    <joint name="${arm_id}_joint_2" type="continuous">
+      <limit effort="0" lower="${radians(-170)}" upper="${radians(170)}" velocity="${radians(465)}" />
+    </joint>
+    <joint name="${arm_id}_joint_2" type="revolute">
       <parent link="${arm_id}_link_1"/>
       <child link="${arm_id}_link_2"/>
       <origin xyz="0 0 0" rpy="0 0 0" />
       <axis xyz="0 1 0" />
-      <!-- <limit effort="100" lower="${radians(-100)}" upper="${radians(145)}" velocity="${radians(310)}" /> -->
-    </joint>
-    <joint name="${arm_id}_joint_3" type="continuous">
+      <limit effort="100" lower="${radians(-110)}" upper="${radians(130)}" velocity="${radians(465)}" />
+    </joint>
+    <joint name="${arm_id}_joint_3" type="revolute">
       <parent link="${arm_id}_link_2"/>
       <child link="${arm_id}_link_3"/>
       <origin xyz="0 0 0.260" rpy="0 0 0" />
       <axis xyz="0 -1 0" />
-      <!-- <limit effort="0" lower="${radians(-70)}" upper="${radians(213)}" velocity="${radians(410)}" /> -->
-    </joint>
-    <joint name="${arm_id}_joint_4" type="continuous">
+      <limit effort="0" lower="${radians(-65)}" upper="${radians(200)}" velocity="${radians(525)}" />
+    </joint>
+    <joint name="${arm_id}_joint_4" type="revolute">
       <parent link="${arm_id}_link_3"/>
       <child link="${arm_id}_link_4"/>
       <origin xyz="0.290 0 0.015" rpy="0 0 0" />
       <axis xyz="-1 0 0" />
-      <!-- <limit effort="0" lower="${radians(-190)}" upper="${radians(190)}" velocity="${radians(550)}" /> -->
-    </joint>
-    <joint name="${arm_id}_joint_5" type="continuous">
+      <limit effort="0" lower="${radians(-200)}" upper="${radians(200)}" velocity="${radians(550)}" />
+    </joint>
+    <joint name="${arm_id}_joint_5" type="revolute">
       <parent link="${arm_id}_link_4"/>
       <child link="${arm_id}_link_5"/>
       <origin xyz="0 0 0" rpy="0 0 0" />
       <axis xyz="0 -1 0" />
-      <!-- <limit effort="0" lower="${radians(-125)}" upper="${radians(125)}" velocity="${radians(545)}" /> -->
-    </joint>
-    <joint name="${arm_id}_joint_6" type="continuous">
+      <limit effort="0" lower="${radians(-123)}" upper="${radians(123)}" velocity="${radians(545)}" />
+    </joint>
+    <joint name="${arm_id}_joint_6" type="revolute">
       <parent link="${arm_id}_link_5"/>
       <child link="${arm_id}_link_6"/>
       <origin xyz="0 0 0" rpy="0 0 0" />
       <axis xyz="-1 0 0" />
-      <!-- <limit effort="0" lower="${radians(-360)}" upper="${radians(360)}" velocity="${radians(1000)}" /> -->
+      <limit effort="0" lower="${radians(-455)}" upper="${radians(455)}" velocity="${radians(1000)}" />
     </joint>
     <link name="${arm_id}_flange"/>

Commit message: removed camera dual arm

File: urdf/single_gp4.xacro (robot description, xacro)
@@ -234,5 +234,5 @@
       </inertial>
     </link>
-    <link name="${arm_id}_link_mountplate">
+    <!-- <link name="${arm_id}_link_mountplate">
     <inertial>
       <origin
@@ -295,5 +295,5 @@
         <origin xyz="0 0 0" rpy="0 0 0"/>
         <geometry>
-          <mesh filename="file://$(find robot_digital_twin)/meshes/eoat/D405_inflated.stl"/>
+          <mesh filename="file://$(find robot_digital_twin)/meshes/eoat/D405.stl"/>
         </geometry>
       </collision>
@@ -311,5 +311,5 @@
         <inertia ixx="1e-6" ixy="0" ixz="0" iyy="1e-6" iyz="0" izz="1e-6" />
       </inertial>
-    </link>
+    </link> -->
     <link name="${arm_id}_link_tool">
     <inertial>
@@ -396,5 +396,5 @@
       <child link="${arm_id}_fts" />
     </joint>
-    <joint name="${arm_id}_fts_plate" type="fixed">
+    <!-- <joint name="${arm_id}_fts_plate" type="fixed">
       <origin xyz="0 0 ${0.0505/2+0.00001}" rpy="${pi/2.0} 0 0" />
       <parent link="${arm_id}_fts" />
@@ -415,7 +415,7 @@
       <parent link="${arm_id}_link_camera" />
       <child link="${arm_id}_link_camera_origin" />
-    </joint>
+    </joint> -->
     <joint name="${arm_id}_fts_tool" type="revolute">
-      <origin xyz="0 0 ${0.0505/2 + 0.00254}" rpy="0 0 ${pi}" />
+      <origin xyz="0 0 ${0.0505/2}" rpy="0 0 ${pi}" />
       <parent link="${arm_id}_fts" />
       <child link="${arm_id}_link_tool" />
