Commit message: cam tilt angle

File: urdf/gp4.xacro (robot description, xacro)
@@ -251,4 +251,59 @@
       </visual>
     </link>
+    <link name="link_precam">
+      <inertial>
+        <mass value="1e-5" />
+        <origin xyz="0 0 0" rpy="0 0 0"/>
+        <inertia ixx="1e-6" ixy="0" ixz="0" iyy="1e-6" iyz="0" izz="1e-6" />
+      </inertial>
+    </link>
+    <link name="link_camera">
+    <inertial>
+      <origin
+        xyz="0 0 0"
+        rpy="0 0 0" />
+      <mass
+        value="0.10811" />
+      <inertia
+        ixx="9.0129E-05"
+        ixy="-1.0891E-08"
+        ixz="9.1598E-09"
+        iyy="9.2026E-05"
+        iyz="-2.749E-07"
+        izz="0.00017818" />
+    </inertial>
+      <visual>
+        <origin xyz="0 0 0" rpy="0 0 0"/>
+        <geometry>
+          <mesh filename="file://$(find robot_digital_twin)/meshes/eoat/tool_camera.stl"/>
+        </geometry>
+        <xacro:material_fanuc_black />
+      </visual>
+      <collision>
+        <origin xyz="0 0 0" rpy="0 0 0"/>
+        <geometry>
+          <mesh filename="file://$(find robot_digital_twin)/meshes/eoat/tool_camera.stl"/>
+        </geometry>
+      </collision>
+    </link>
+    <link name="link_camera_origin">
+    <collision>
+      <origin xyz="0 0 0" rpy="0 0 0"/>
+      <geometry>
+        <box size="0.0001 0.0001 0.0001"/>
+      </geometry>
+    </collision>
+    <visual>
+      <origin xyz="0 0 0" rpy="0 0 0"/>
+      <geometry>
+        <box size="0.0001 0.01 0.01"/>
+      </geometry>
+    </visual>
+      <inertial>
+        <mass value="1e-5" />
+        <origin xyz="0 0 0" rpy="0 0 0"/>
+        <inertia ixx="1e-6" ixy="0" ixz="0" iyy="1e-6" iyz="0" izz="1e-6" />
+      </inertial>
+    </link>
     <!-- joints: main serial chain -->
     <joint name="joint_1" type="continuous">
@@ -313,7 +368,12 @@
       <limit velocity="0" effort="0" lower="0" upper="0" />
     </joint>
-    <!-- <joint name="tool_camera" type="fixed">
-      <origin xyz="0 -0.04625 0.028" rpy="${-pi/2.0} ${-pi/2.0} ${pi}" />
+    <joint name="tool_precam" type="fixed">
+      <origin xyz="0 -0.04625 0.028" rpy="${pi/2} -${pi/2}  0" />
       <parent link="link_tool" />
+      <child link="link_precam" />
+    </joint>
+    <joint name="precam_camera" type="fixed">
+      <origin xyz="0 0 0" rpy="0 ${pi*0.4} 0" />
+      <parent link="link_precam" />
       <child link="link_camera" />
     </joint>
@@ -322,5 +382,5 @@
       <parent link="link_camera" />
       <child link="link_camera_origin" />
-    </joint> -->
+    </joint>
   </xacro:macro>
   <xacro:Yaskawa_gp4>
@@ -369,4 +429,40 @@
       </plugin>
   </gazebo>
+  <gazebo reference="link_camera_origin">
+  <sensor name="$depth_camera" type="depth">
+    <update_rate>30</update_rate>
+    <camera>
+      <horizontal_fov>1.22173</horizontal_fov> <!-- 70deg -->
+      <image>
+        <width>1920</width>
+        <height>1080</height>
+        <format>R8G8B8</format>
+      </image>
+      <clip>
+        <near>0.01</near>
+        <far>2</far>
+      </clip>
+    </camera>
+    <plugin name="$depth_camera_controller" filename="libgazebo_ros_openni_kinect.so">
+      <baseline>0.2</baseline>
+      <alwaysOn>true</alwaysOn>
+      <updateRate>0</updateRate>
+      <cameraName>wrist_camera</cameraName>
+      <frameName>depth_camera_link</frameName>
+      <pointCloudCutoff>0.005</pointCloudCutoff>
+      <pointCloudCutoffMax>2.0</pointCloudCutoffMax>
+      <distortionK1>0</distortionK1>
+      <distortionK2>0</distortionK2>
+      <distortionK3>0</distortionK3>
+      <distortionT1>0</distortionT1>
+      <distortionT2>0</distortionT2>
+      <CxPrime>0</CxPrime>
+      <Cx>0</Cx>
+      <Cy>0</Cy>
+      <focalLength>0</focalLength>
+      <hackBaseline>0</hackBaseline>
+    </plugin>
+  </sensor>
+</gazebo>
   <gazebo reference="base">
      <material>Gazebo/Blue</material>

Commit message: add mfi

File: urdf/gp4.xacro (robot description, xacro)
@@ -246,5 +246,5 @@
         <origin xyz="0 0 0" rpy="0 0 0"/>
         <geometry>
-          <mesh filename="file://$(find robot_digital_twin)/meshes/eoat/tool_base.stl"/>
+          <mesh filename="file://$(find robot_digital_twin)/meshes/eoat/tool_base_tilt.stl"/>
         </geometry>
         <xacro:material_yaskawa_silver />
@@ -369,10 +369,10 @@
     </joint>
     <joint name="tool_precam" type="fixed">
-      <origin xyz="0 -0.04625 0.028" rpy="${pi/2} -${pi/2}  0" />
+      <origin xyz="0 -0.06767 0.01651" rpy="${pi/2} -${pi/2}  0" />
       <parent link="link_tool" />
       <child link="link_precam" />
     </joint>
     <joint name="precam_camera" type="fixed">
-      <origin xyz="0 0 0" rpy="0 ${pi*0.4} 0" />
+      <origin xyz="0 0 0" rpy="0 ${pi*40/180} 0" />
       <parent link="link_precam" />
       <child link="link_camera" />
@@ -440,5 +440,5 @@
       </image>
       <clip>
-        <near>0.01</near>
+        <near>0.005</near>
         <far>2</far>
       </clip>

Commit message: new tool

File: urdf/gp4.xacro (robot description, xacro)
@@ -369,10 +369,10 @@
     </joint>
     <joint name="tool_precam" type="fixed">
-      <origin xyz="0 -0.06767 0.01651" rpy="${pi/2} -${pi/2}  0" />
+      <origin xyz="0 -0.062194148 -0.005909903" rpy="${pi/2} -${pi/2}  0" />
       <parent link="link_tool" />
       <child link="link_precam" />
     </joint>
     <joint name="precam_camera" type="fixed">
-      <origin xyz="0 0 0" rpy="0 ${pi*40/180} 0" />
+      <origin xyz="0 0 0" rpy="0 ${pi*45/180} 0" />
       <parent link="link_precam" />
       <child link="link_camera" />

Commit message: update simulator, controller and collision-checker with moveit

File: urdf/gp4.xacro (robot description, xacro)
@@ -2,22 +2,29 @@
 <robot
   name="Yaskawa_gp4" xmlns:xacro="http://ros.org/wiki/xacro">
-  <xacro:macro name="Yaskawa_gp4">
+  <xacro:macro name="Yaskawa_gp4" params="arm_id:='gp4' description_pkg:='robot_digital_twin' connected_to:='' xyz:='0 0 0' rpy:='0 0 0'">
   <xacro:include
     filename="$(find robot_digital_twin)/urdf/common_materials.xacro"/>
-  <link name = "world"/>
-  <joint name = "world_fixed"
-    type = "fixed">
-    <parent link = "world" />
-    <child link = "base" />
+  <xacro:if value="${connected_to == ''}">
+    <link name="world" />
+    <xacro:property name="base_frame_name" value="world"/>
+  </xacro:if>
+  <xacro:unless value="${connected_to == ''}">
+    <xacro:property name="base_frame_name" value="${connected_to}"/>
+  </xacro:unless>
+  <joint name="${arm_id}_to_${base_frame_name}" type="fixed">
+      <parent link="${base_frame_name}"/>
+      <child link="${arm_id}_base"/>
+      <origin rpy="${rpy}" xyz="${xyz}"/>
+      <dynamics damping="1.0"/>
   </joint>
   <!-- ROS-Industrial 'base' frame: base_link to gp4 World Coordinates transform -->
-    <link name="base" />
-    <joint name="base_link-base" type="fixed">
+    <link name="${arm_id}_base" />
+    <joint name="${arm_id}_base_link-base" type="fixed">
       <origin xyz="0 0 0.0" rpy="0 0 0"/>
-      <parent link="base"/>
-      <child link="base_link"/>
+      <parent link="${arm_id}_base"/>
+      <child link="${arm_id}_base_link"/>
     </joint>
     <!-- links: main serial chain -->
-    <link name="base_link">
+    <link name="${arm_id}_base_link">
      <inertial>
       <origin
@@ -46,5 +53,5 @@
       </collision>
     </link>
-    <link name="link_1">
+    <link name="${arm_id}_link_1">
     <inertial>
       <origin
@@ -73,5 +80,5 @@
       </collision>
     </link>
-    <link name="link_2">
+    <link name="${arm_id}_link_2">
     <inertial>
       <origin
@@ -100,5 +107,5 @@
       </collision>
     </link>
-    <link name="link_3">
+    <link name="${arm_id}_link_3">
     <inertial>
       <origin
@@ -127,5 +134,5 @@
       </collision>
     </link>
-    <link name="link_4">
+    <link name="${arm_id}_link_4">
     <inertial>
       <origin
@@ -154,5 +161,5 @@
       </collision>
     </link>
-    <link name="link_5">
+    <link name="${arm_id}_link_5">
     <inertial>
       <origin
@@ -181,5 +188,5 @@
       </collision>
     </link>
-    <link name="link_6">
+    <link name="${arm_id}_link_6">
     <inertial>
       <origin
@@ -208,5 +215,5 @@
       </collision>
     </link>
-    <link name="fts">
+    <link name="${arm_id}_fts">
       <collision>
         <origin xyz="0 0 0" rpy=" 0 0 0"/>
@@ -228,5 +235,5 @@
       </inertial>
     </link>
-    <link name="link_tool">
+    <link name="${arm_id}_link_tool">
     <inertial>
       <origin
@@ -243,4 +250,10 @@
         izz="0.00017818" />
     </inertial>
+    <collision>
+      <origin xyz="0 0 0" rpy="0 0 0"/>
+      <geometry>
+        <mesh filename="file://$(find robot_digital_twin)/meshes/eoat/tool_base_tilt.stl"/>
+      </geometry>
+    </collision>
       <visual>
         <origin xyz="0 0 0" rpy="0 0 0"/>
@@ -251,5 +264,5 @@
       </visual>
     </link>
-    <link name="link_precam">
+    <link name="${arm_id}_link_precam">
       <inertial>
         <mass value="1e-5" />
@@ -258,5 +271,5 @@
       </inertial>
     </link>
-    <link name="link_camera">
+    <link name="${arm_id}_link_camera">
     <inertial>
       <origin
@@ -287,5 +300,5 @@
       </collision>
     </link>
-    <link name="link_camera_origin">
+    <link name="${arm_id}_link_camera_origin">
     <collision>
       <origin xyz="0 0 0" rpy="0 0 0"/>
@@ -307,7 +320,7 @@
     </link>
     <!-- joints: main serial chain -->
-    <joint name="joint_1" type="continuous">
-      <parent link="base_link"/>
-      <child link="link_1"/>
+    <joint name="${arm_id}_joint_1" type="continuous">
+      <parent link="${arm_id}_base_link"/>
+      <child link="${arm_id}_link_1"/>
       <origin xyz="0 0 0.330" rpy="0 0 0" />
       <axis xyz="0 0 1" />
@@ -315,197 +328,191 @@
       <!-- <limit effort="0" lower="${radians(-170)}" upper="${radians(170)}" velocity="${radians(370)}" /> -->
     </joint>
-    <joint name="joint_2" type="continuous">
-      <parent link="link_1"/>
-      <child link="link_2"/>
+    <joint name="${arm_id}_joint_2" type="continuous">
+      <parent link="${arm_id}_link_1"/>
+      <child link="${arm_id}_link_2"/>
       <origin xyz="0 0 0" rpy="0 0 0" />
       <axis xyz="0 1 0" />
       <!-- <limit effort="100" lower="${radians(-100)}" upper="${radians(145)}" velocity="${radians(310)}" /> -->
     </joint>
-    <joint name="joint_3" type="continuous">
-      <parent link="link_2"/>
-      <child link="link_3"/>
+    <joint name="${arm_id}_joint_3" type="continuous">
+      <parent link="${arm_id}_link_2"/>
+      <child link="${arm_id}_link_3"/>
       <origin xyz="0 0 0.260" rpy="0 0 0" />
       <axis xyz="0 -1 0" />
       <!-- <limit effort="0" lower="${radians(-70)}" upper="${radians(213)}" velocity="${radians(410)}" /> -->
     </joint>
-    <joint name="joint_4" type="continuous">
-      <parent link="link_3"/>
-      <child link="link_4"/>
+    <joint name="${arm_id}_joint_4" type="continuous">
+      <parent link="${arm_id}_link_3"/>
+      <child link="${arm_id}_link_4"/>
       <origin xyz="0.290 0 0.015" rpy="0 0 0" />
       <axis xyz="-1 0 0" />
       <!-- <limit effort="0" lower="${radians(-190)}" upper="${radians(190)}" velocity="${radians(550)}" /> -->
     </joint>
-    <joint name="joint_5" type="continuous">
-      <parent link="link_4"/>
-      <child link="link_5"/>
+    <joint name="${arm_id}_joint_5" type="continuous">
+      <parent link="${arm_id}_link_4"/>
+      <child link="${arm_id}_link_5"/>
       <origin xyz="0 0 0" rpy="0 0 0" />
       <axis xyz="0 -1 0" />
       <!-- <limit effort="0" lower="${radians(-125)}" upper="${radians(125)}" velocity="${radians(545)}" /> -->
     </joint>
-    <joint name="joint_6" type="continuous">
-      <parent link="link_5"/>
-      <child link="link_6"/>
+    <joint name="${arm_id}_joint_6" type="continuous">
+      <parent link="${arm_id}_link_5"/>
+      <child link="${arm_id}_link_6"/>
       <origin xyz="0 0 0" rpy="0 0 0" />
       <axis xyz="-1 0 0" />
       <!-- <limit effort="0" lower="${radians(-360)}" upper="${radians(360)}" velocity="${radians(1000)}" /> -->
     </joint>
-    <link name="flange"/>
-    <joint name="joint_6_t-flange" type="fixed">
+    <link name="${arm_id}_flange"/>
+    <joint name="${arm_id}_joint_6_t-flange" type="fixed">
       <origin xyz="0.072 0 0" rpy="0 0 0"/>
-      <parent link="link_6"/>
-      <child link="flange"/>
-    </joint>
-    <joint name="link_6_fts" type="fixed">
+      <parent link="${arm_id}_link_6"/>
+      <child link="${arm_id}_flange"/>
+    </joint>
+    <joint name="${arm_id}_link_6_fts" type="fixed">
       <origin xyz="${0.0505/2} 0 0" rpy="0 ${pi/2.0} 0" />
-      <parent link="flange" />
-      <child link="fts" />
-    </joint>
-    <joint name="fts_tool" type="revolute">
+      <parent link="${arm_id}_flange" />
+      <child link="${arm_id}_fts" />
+    </joint>
+    <joint name="${arm_id}_fts_tool" type="revolute">
       <origin xyz="0 0 ${0.0505/2}" rpy="0 0 ${pi}" />
-      <parent link="fts" />
-      <child link="link_tool" />
+      <parent link="${arm_id}_fts" />
+      <child link="${arm_id}_link_tool" />
       <axis xyz="0 0 1" />
       <limit velocity="0" effort="0" lower="0" upper="0" />
     </joint>
-    <joint name="tool_precam" type="fixed">
+    <joint name="${arm_id}_tool_precam" type="fixed">
       <origin xyz="0 -0.062194148 -0.005909903" rpy="${pi/2} -${pi/2}  0" />
-      <parent link="link_tool" />
-      <child link="link_precam" />
-    </joint>
-    <joint name="precam_camera" type="fixed">
+      <parent link="${arm_id}_link_tool" />
+      <child link="${arm_id}_link_precam" />
+    </joint>
+    <joint name="${arm_id}_precam_camera" type="fixed">
       <origin xyz="0 0 0" rpy="0 ${pi*45/180} 0" />
-      <parent link="link_precam" />
-      <child link="link_camera" />
-    </joint>
-    <joint name="camera_imgplane" type="fixed">
+      <parent link="${arm_id}_link_precam" />
+      <child link="${arm_id}_link_camera" />
+    </joint>
+    <joint name="${arm_id}_camera_imgplane" type="fixed">
       <origin xyz="0.013 0.0 0.0305" rpy="0 0 0" />
-      <parent link="link_camera" />
-      <child link="link_camera_origin" />
+      <parent link="${arm_id}_link_camera" />
+      <child link="${arm_id}_link_camera_origin" />
     </joint>
   </xacro:macro>
-  <xacro:Yaskawa_gp4>
-  </xacro:Yaskawa_gp4>
-  <xacro:macro name="transmission_block" params="joint_name">
-    <transmission name = "trans_${joint_name}">
-      <type>transmission_interface/SimpleTransmission</type>
-      <joint name = "${joint_name}">
-        <hardwareInterface>hardware_interface/PositionJointInterface</hardwareInterface>
-      </joint>
-      <actuator name = "${joint_name}_motor">
-        <hardwareInterface>hardware_interface/PositionJointInterface</hardwareInterface>
-        <mechanicalReduction>1</mechanicalReduction>
-      </actuator>
-    </transmission>
+  <xacro:macro name="gp4_gazebo" params="arm_id:='gp4'">
+    <xacro:macro name="transmission_block" params="joint_name">
+      <transmission name = "trans_${joint_name}">
+        <type>transmission_interface/SimpleTransmission</type>
+        <joint name = "${joint_name}">
+          <hardwareInterface>hardware_interface/PositionJointInterface</hardwareInterface>
+        </joint>
+        <actuator name = "${joint_name}_motor">
+          <hardwareInterface>hardware_interface/PositionJointInterface</hardwareInterface>
+          <mechanicalReduction>1</mechanicalReduction>
+        </actuator>
+      </transmission>
+    </xacro:macro>
+    <!-- transmission block-->
+    <xacro:transmission_block joint_name = "${arm_id}_joint_1"/>
+    <xacro:transmission_block joint_name = "${arm_id}_joint_2"/>
+    <xacro:transmission_block joint_name = "${arm_id}_joint_3"/>
+    <xacro:transmission_block joint_name = "${arm_id}_joint_4"/>
+    <xacro:transmission_block joint_name = "${arm_id}_joint_5"/>
+    <xacro:transmission_block joint_name = "${arm_id}_joint_6"/>
+    <gazebo reference="fts_tool">
+        <provideFeedback>true</provideFeedback>
+    </gazebo>
+    <gazebo>
+      <provideFeedback>true</provideFeedback>
+        <plugin name="ft_sensor" filename="libgazebo_ros_ft_sensor.so">
+            <!-- <robotNamespace>/gp4_gazebo</robotNamespace> -->
+            <alwaysOn> true </alwaysOn>
+            <updateRate>125.0</updateRate>
+            <topicName>${arm_id}_ft_sensor</topicName>
+            <jointName>${arm_id}_fts_tool</jointName>
+            <noise>
+              <type>gaussian</type>
+              <mean>0.0</mean>
+              <stddev>0.001</stddev>
+            </noise>
+        </plugin>
+    </gazebo>
+    <gazebo reference="link_camera_origin">
+    <sensor name="$depth_camera" type="depth">
+      <update_rate>30</update_rate>
+      <camera>
+        <horizontal_fov>1.22173</horizontal_fov> <!-- 70deg -->
+        <image>
+          <width>1920</width>
+          <height>1080</height>
+          <format>R8G8B8</format>
+        </image>
+        <clip>
+          <near>0.005</near>
+          <far>2</far>
+        </clip>
+      </camera>
+      <plugin name="$depth_camera_controller" filename="libgazebo_ros_openni_kinect.so">
+        <baseline>0.2</baseline>
+        <alwaysOn>true</alwaysOn>
+        <updateRate>0</updateRate>
+        <cameraName>${arm_id}_wrist_camera</cameraName>
+        <frameName>${arm_id}_depth_camera_link</frameName>
+        <pointCloudCutoff>0.005</pointCloudCutoff>
+        <pointCloudCutoffMax>2.0</pointCloudCutoffMax>
+        <distortionK1>0</distortionK1>
+        <distortionK2>0</distortionK2>
+        <distortionK3>0</distortionK3>
+        <distortionT1>0</distortionT1>
+        <distortionT2>0</distortionT2>
+        <CxPrime>0</CxPrime>
+        <Cx>0</Cx>
+        <Cy>0</Cy>
+        <focalLength>0</focalLength>
+        <hackBaseline>0</hackBaseline>
+      </plugin>
+    </sensor>
+  </gazebo>
+    <gazebo reference="${arm_id}_base">
+      <material>Gazebo/Blue</material>
+      <visual> <transparency> 0 </transparency> </visual>
+    </gazebo>
+    <gazebo reference="${arm_id}_base_link">
+      <material>Gazebo/Blue</material>
+      <visual> <transparency> 0 </transparency> </visual>
+    </gazebo>
+    <gazebo reference="${arm_id}_link_1">
+      <material>Gazebo/Blue</material>
+      <visual> <transparency> 0 </transparency> </visual>
+    </gazebo>
+    <gazebo reference="${arm_id}_link_2">
+      <material>Gazebo/Blue</material>
+      <visual> <transparency> 0 </transparency> </visual>
+    </gazebo>
+    <gazebo reference="${arm_id}_link_3">
+      <material>Gazebo/Blue</material>
+      <visual> <transparency> 0 </transparency> </visual>
+    </gazebo>
+    <gazebo reference="${arm_id}_link_4">
+      <material>Gazebo/Blue</material>
+      <visual> <transparency> 0 </transparency> </visual>
+    </gazebo>
+    <gazebo reference="${arm_id}_link_5">
+      <material>Gazebo/Blue</material>
+      <visual> <transparency> 0 </transparency> </visual>
+    </gazebo>
+    <gazebo reference="${arm_id}_link_6">
+      <material>Gazebo/Black</material>
+      <visual> <transparency> 0 </transparency> </visual>
+    </gazebo>
+    <gazebo reference="${arm_id}_link_tool">
+      <material>Gazebo/Black</material>
+      <visual> <transparency> 0 </transparency> </visual>
+    </gazebo>
+    <gazebo reference="${arm_id}_fts">
+      <material>Gazebo/Black</material>
+      <visual> <transparency> 0 </transparency> </visual>
+    </gazebo>
+    <gazebo reference="${arm_id}_link_camera_origin">
+      <material>Gazebo/Black</material>
+      <visual> <transparency> 0 </transparency> </visual>
+    </gazebo>
   </xacro:macro>
-  <xacro:transmission_block joint_name = "joint_1"/>
-  <xacro:transmission_block joint_name = "joint_2"/>
-  <xacro:transmission_block joint_name = "joint_3"/>
-  <xacro:transmission_block joint_name = "joint_4"/>
-  <xacro:transmission_block joint_name = "joint_5"/>
-  <xacro:transmission_block joint_name = "joint_6"/>
-  <gazebo>
-    <plugin name="gazebo_ros_control" filename="libgazebo_ros_control.so">
-	    <!-- <robotNamespace>/gp4_gazebo</robotNamespace> -->
-      <robotSimType>gazebo_ros_control/DefaultRobotHWSim</robotSimType>
-      <legacyModeNS>true</legacyModeNS>
-    </plugin>
-  </gazebo>
-  <gazebo reference="fts_tool">
-      <provideFeedback>true</provideFeedback>
-  </gazebo>
-  <gazebo>
-    <provideFeedback>true</provideFeedback>
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
Commit message: update

File: urdf/gp4.xacro (robot description, xacro)
@@ -212,11 +212,11 @@
         <origin xyz="0 0 0" rpy=" 0 0 0"/>
         <geometry>
-          <cylinder length="0.041" radius="0.035"/>
-        </geometry>
-      </collision>
-      <visual>
-        <origin xyz="0 0 0" rpy="0 0 0"/>
-        <geometry>
-          <cylinder length="0.041" radius="0.035"/>
+          <cylinder length="0.0505" radius="0.035"/>
+        </geometry>
+      </collision>
+      <visual>
+        <origin xyz="0 0 0" rpy="0 0 0"/>
+        <geometry>
+          <cylinder length="0.0505" radius="0.035"/>
         </geometry>
         <xacro:material_yaskawa_silver />

Commit message: rm cam

File: urdf/gp4.xacro (robot description, xacro)
@@ -228,5 +228,5 @@
       </inertial>
     </link>
-    <link name="link_mountplate">
+    <!-- <link name="link_mountplate">
     <inertial>
       <origin
@@ -305,5 +305,5 @@
         <inertia ixx="1e-6" ixy="0" ixz="0" iyy="1e-6" iyz="0" izz="1e-6" />
       </inertial>
-    </link>
+    </link> -->
     <link name="link_tool">
     <inertial>
@@ -384,5 +384,5 @@
       <child link="fts" />
     </joint>
-    <joint name="fts_plate" type="revolute">
+    <!-- <joint name="fts_plate" type="revolute">
       <origin xyz="0 0 ${0.0505/2+0.00001}" rpy="${pi/2.0} 0 0" />
       <parent link="fts" />
@@ -405,7 +405,8 @@
       <parent link="link_camera" />
       <child link="link_camera_origin" />
-    </joint>
+    </joint> -->
     <joint name="fts_tool" type="revolute">
-      <origin xyz="0 0 ${0.0505/2 + 0.00254}" rpy="0 0 ${pi}" />
+      <!-- <origin xyz="0 0 ${0.0505/2 + 0.00254}" rpy="0 0 ${pi}" /> -->
+      <origin xyz="0 0 ${0.0505/2}" rpy="0 0 ${pi}" />
       <parent link="fts" />
       <child link="link_tool" />
@@ -459,5 +460,5 @@
       </plugin>
   </gazebo>
-  <gazebo reference="link_camera_origin">
+  <!-- <gazebo reference="link_camera_origin">
   <sensor name="$depth_camera" type="depth">
     <update_rate>30</update_rate>
@@ -494,5 +495,5 @@
     </plugin>
   </sensor>
-</gazebo>
+</gazebo> -->
   <gazebo reference="base">
      <material>Gazebo/Blue</material>
