Commit message: update lego eoat with gen 3

File: urdf/gp4.xacro (robot description, xacro)
@@ -324,5 +324,5 @@
         <origin xyz="0 0 0" rpy="0 0 0"/>
         <geometry>
-          <mesh filename="file://$(find robot_digital_twin)/meshes/eoat/tool.stl"/>
+          <mesh filename="file://$(find robot_digital_twin)/meshes/eoat/tool_with_cam.stl"/>
         </geometry>
         <xacro:material_yaskawa_silver />

File: urdf/single_gp4.xacro (robot description, xacro)
@@ -330,5 +330,5 @@
       <origin xyz="0 0 0" rpy="0 0 0"/>
       <geometry>
-        <mesh filename="file://$(find robot_digital_twin)/meshes/eoat/tool.stl"/>
+        <mesh filename="file://$(find robot_digital_twin)/meshes/eoat/tool_with_cam.stl"/>
       </geometry>
     </collision>
@@ -336,5 +336,5 @@
         <origin xyz="0 0 0" rpy="0 0 0"/>
         <geometry>
-          <mesh filename="file://$(find robot_digital_twin)/meshes/eoat/tool.stl"/>
+          <mesh filename="file://$(find robot_digital_twin)/meshes/eoat/tool_with_cam.stl"/>
         </geometry>
         <xacro:material_yaskawa_silver />
