Commit message: update the newest version

File: urdf/bolt.xacro (robot description, xacro)
@@ -54,5 +54,5 @@
   </link>
   <gazebo reference="bolt">
-  <kinematic>0</kinematic>
+  <kinematic>1</kinematic>
   <xacro:if value="${color == 'Orange'}">
      <material>Gazebo/Orange</material>

File: urdf/cc_block.xacro (robot description, xacro)
@@ -6,4 +6,5 @@
   <xacro:property name="scale" value="0.001"/>
   <xacro:property name="color" value="$(arg cc_block_color)"/>
+  <xacro:property name="enable_dynamics" value="false"/>
   <link
     name="cc_block">
@@ -22,5 +23,5 @@
         izz="0.00005" />
       </inertial> -->
-      <mass
+       <mass
         value="0.0001" />
       <inertia
@@ -46,20 +47,5 @@
       </material>
     </visual>
-    <collision>
-      <origin
-        xyz="0 0 0"
-        rpy="0 0 0" />
-      <geometry>
-        <mesh scale="${scale} ${scale} ${scale}"
-          filename="file://$(find robot_digital_twin)/meshes/share_parts/cc_block.STL"/>
-      </geometry>
-      <gazebo>
-        <mu>100000.0</mu>        <!-- Lateral friction coefficient -->
-        <mu2>100000.0</mu2>      <!-- Second friction coefficient for anisotropic friction -->
-        <kp>100000</kp>     <!-- Spring coefficient (stiffness) -->
-        <kd>1</kd>          <!-- Damping coefficient -->
-      </gazebo>
-    </collision>
-    <gravity>1</gravity>
+    <gravity>0</gravity>
   </link>
   <gazebo reference="cc_block">

File: urdf/nut.xacro (robot description, xacro)
@@ -54,5 +54,5 @@
   </link>
   <gazebo reference="nut">
-  <kinematic>0</kinematic>
+  <kinematic>1</kinematic>
   <xacro:if value="${color == 'Orange'}">
      <material>Gazebo/Orange</material>

File: urdf/rr_block.xacro (robot description, xacro)
@@ -51,5 +51,5 @@
       </gazebo>
     </collision>
-    <gravity>1</gravity>
+    <gravity>0</gravity>
   </link>
   <gazebo reference="rr_block">
