Commit message: new tool

File: urdf/camera.xacro (robot description, xacro)
@@ -32,5 +32,5 @@
         <origin xyz="0 0 0" rpy="0 0 0"/>
         <geometry>
-          <mesh filename="file://$(find robot_digital_twin)/meshes/eoat/tool_camera.stl"/>
+          <mesh filename="file://$(find robot_digital_twin)/meshes/eoat/L515.stl"/>
         </geometry>
         <xacro:material_fanuc_black />
@@ -39,5 +39,5 @@
         <origin xyz="0 0 0" rpy="0 0 0"/>
         <geometry>
-          <mesh filename="file://$(find robot_digital_twin)/meshes/eoat/tool_camera.stl"/>
+          <mesh filename="file://$(find robot_digital_twin)/meshes/eoat/L515.stl"/>
         </geometry>
       </collision>

File: urdf/fanuc_arm.xacro (robot description, xacro)
@@ -295,5 +295,5 @@
         <origin xyz="0 0 0" rpy="0 0 0"/>
         <geometry>
-          <mesh filename="file://$(find robot_digital_twin)/meshes/eoat/tool_camera.stl"/>
+          <mesh filename="file://$(find robot_digital_twin)/meshes/eoat/L515.stl"/>
         </geometry>
         <xacro:material_fanuc_black />
@@ -302,5 +302,5 @@
         <origin xyz="0 0 0" rpy="0 0 0"/>
         <geometry>
-          <mesh filename="file://$(find robot_digital_twin)/meshes/eoat/tool_camera.stl"/>
+          <mesh filename="file://$(find robot_digital_twin)/meshes/eoat/L515.stl"/>
         </geometry>
       </collision>

File: urdf/gp4.xacro (robot description, xacro)
@@ -228,5 +228,5 @@
       </inertial>
     </link>
-    <link name="link_tool">
+    <link name="link_mountplate">
     <inertial>
       <origin
@@ -246,8 +246,14 @@
         <origin xyz="0 0 0" rpy="0 0 0"/>
         <geometry>
-          <mesh filename="file://$(find robot_digital_twin)/meshes/eoat/tool_base.stl"/>
+          <mesh filename="file://$(find robot_digital_twin)/meshes/eoat/D405_mount.stl"/>
         </geometry>
         <xacro:material_yaskawa_silver />
       </visual>
+      <collision>
+        <origin xyz="0 0 0" rpy="0 0 0"/>
+        <geometry>
+          <mesh filename="file://$(find robot_digital_twin)/meshes/eoat/D405_mount.stl"/>
+        </geometry>
+      </collision>
     </link>
     <link name="link_precam">
@@ -276,5 +282,5 @@
         <origin xyz="0 0 0" rpy="0 0 0"/>
         <geometry>
-          <mesh filename="file://$(find robot_digital_twin)/meshes/eoat/tool_camera.stl"/>
+          <mesh filename="file://$(find robot_digital_twin)/meshes/eoat/D405.stl"/>
         </geometry>
         <xacro:material_fanuc_black />
@@ -283,19 +289,13 @@
         <origin xyz="0 0 0" rpy="0 0 0"/>
         <geometry>
-          <mesh filename="file://$(find robot_digital_twin)/meshes/eoat/tool_camera.stl"/>
+          <mesh filename="file://$(find robot_digital_twin)/meshes/eoat/D405.stl"/>
         </geometry>
       </collision>
     </link>
     <link name="link_camera_origin">
-    <collision>
-      <origin xyz="0 0 0" rpy="0 0 0"/>
-      <geometry>
-        <box size="0.0001 0.0001 0.0001"/>
-      </geometry>
-    </collision>
     <visual>
       <origin xyz="0 0 0" rpy="0 0 0"/>
       <geometry>
-        <box size="0.0001 0.01 0.01"/>
+        <box size="0.0001 0.002 0.001"/>
       </geometry>
     </visual>
@@ -305,4 +305,27 @@
         <inertia ixx="1e-6" ixy="0" ixz="0" iyy="1e-6" iyz="0" izz="1e-6" />
       </inertial>
+    </link>
+    <link name="link_tool">
+    <inertial>
+      <origin
+        xyz="0 0 0"
+        rpy="0 0 0" />
+      <mass
+        value="0.10811" />
+      <inertia
+        ixx="9.0129E-05"
+        ixy="-1.0891E-08"
+        ixz="9.1598E-09"
+        iyy="9.2026E-05"
+        iyz="-2.749E-07"
+        izz="0.00017818" />
+    </inertial>
+      <visual>
+        <origin xyz="0 0 0" rpy="0 0 0"/>
+        <geometry>
+          <mesh filename="file://$(find robot_digital_twin)/meshes/eoat/tool.stl"/>
+        </geometry>
+        <xacro:material_yaskawa_silver />
+      </visual>
     </link>
     <!-- joints: main serial chain -->
@@ -361,25 +384,32 @@
       <child link="fts" />
     </joint>
+    <joint name="fts_plate" type="revolute">
+      <origin xyz="0 0 ${0.0505/2+0.00001}" rpy="${pi/2.0} 0 0" />
+      <parent link="fts" />
+      <child link="link_mountplate" />
+      <axis xyz="0 0 1" />
+      <limit velocity="0" effort="0" lower="0" upper="0" />
+    </joint>
+    <joint name="plate_precam" type="fixed">
+      <origin xyz="0 0 0" rpy="-${pi/2.0} 0  0" />
+      <parent link="link_mountplate" />
+      <child link="link_precam" />
+    </joint>
+    <joint name="precam_camera" type="fixed">
+      <origin xyz="0 0.053512 ${0.00254+0.023+0.00001}" rpy="0  0  0" />
+      <parent link="link_precam" />
+      <child link="link_camera" />
+    </joint>
+    <joint name="camera_imgplane" type="fixed">
+      <origin xyz="0.009 0 0" rpy="0 ${pi/2 + pi} -${pi/2}" />
+      <parent link="link_camera" />
+      <child link="link_camera_origin" />
+    </joint>
     <joint name="fts_tool" type="revolute">
-      <origin xyz="0 0 ${0.0505/2}" rpy="0 0 ${pi}" />
+      <origin xyz="0 0 ${0.0505/2 + 0.00254}" rpy="0 0 ${pi}" />
       <parent link="fts" />
       <child link="link_tool" />
       <axis xyz="0 0 1" />
       <limit velocity="0" effort="0" lower="0" upper="0" />
-    </joint>
-    <joint name="tool_precam" type="fixed">
-      <origin xyz="0 -0.062194148 -0.005909903" rpy="${pi/2} -${pi/2}  0" />
-      <parent link="link_tool" />
-      <child link="link_precam" />
-    </joint>
-    <joint name="precam_camera" type="fixed">
-      <origin xyz="0 0 0" rpy="0 ${pi*45/180} 0" />
-      <parent link="link_precam" />
-      <child link="link_camera" />
-    </joint>
-    <joint name="camera_imgplane" type="fixed">
-      <origin xyz="0.013 0.0 0.0305" rpy="0 0 0" />
-      <parent link="link_camera" />
-      <child link="link_camera_origin" />
     </joint>
   </xacro:macro>
@@ -433,5 +463,5 @@
     <update_rate>30</update_rate>
     <camera>
-      <horizontal_fov>1.22173</horizontal_fov> <!-- 70deg -->
+      <horizontal_fov>1.22173</horizontal_fov>
       <image>
         <width>1920</width>

Commit message: reposition camera

File: urdf/camera.xacro (robot description, xacro)
@@ -64,5 +64,5 @@
     <!-- joints: main serial chain -->
     <joint name="precam_camera" type="fixed">
-      <origin xyz="0 0 0" rpy="0 ${pi*45/180} 0" />
+      <origin xyz="0 0 0" rpy="0 0 0" />
       <parent link="base" />
       <child link="link_camera" />

Commit message: add two orbbec camera

File: urdf/camera.xacro (robot description, xacro)
@@ -32,5 +32,5 @@
         <origin xyz="0 0 0" rpy="0 0 0"/>
         <geometry>
-          <mesh filename="file://$(find robot_digital_twin)/meshes/eoat/L515.stl"/>
+          <mesh filename="file://$(find robot_digital_twin)/meshes/eoat/femto_bolt.stl"/>
         </geometry>
         <xacro:material_fanuc_black />
@@ -39,5 +39,5 @@
         <origin xyz="0 0 0" rpy="0 0 0"/>
         <geometry>
-          <mesh filename="file://$(find robot_digital_twin)/meshes/eoat/L515.stl"/>
+          <mesh filename="file://$(find robot_digital_twin)/meshes/eoat/femto_bolt.stl"/>
         </geometry>
       </collision>
@@ -69,5 +69,5 @@
     </joint>
     <joint name="camera_imgplane" type="fixed">
-      <origin xyz="0.013 0.0 0.0305" rpy="0 0 0" />
+      <origin xyz="0.045 0 0" rpy="0 0 0" />
       <parent link="link_camera" />
       <child link="link_camera_origin" />
@@ -80,8 +80,8 @@
     <update_rate>30</update_rate>
     <camera>
-      <horizontal_fov>1.22173</horizontal_fov> <!-- 70deg -->
+      <horizontal_fov>1.39626340156</horizontal_fov> <!-- 80deg -->
       <image>
-        <width>1920</width>
-        <height>1080</height>
+        <width>3840</width>
+        <height>2160</height>
         <format>R8G8B8</format>
       </image>
@@ -95,5 +95,5 @@
       <alwaysOn>true</alwaysOn>
       <updateRate>0</updateRate>
-      <cameraName>wrist_camera</cameraName>
+      <cameraName>fixed_camera</cameraName>
       <frameName>depth_camera_link</frameName>
       <pointCloudCutoff>0.005</pointCloudCutoff>
