Commit message: update the parameters

File: config/gazebo_dual_gp4.urdf (robot description, URDF)
Before this commit: robot dual_gp4, 30 links, 29 joints
Joints:
- joint left_arm_to_base: origin xyz=-0.6 0 1 rpy=0 0 0 -> xyz=0 0 0 rpy=0 0 0
- joint right_arm_to_base: origin xyz=0.6 0 1 rpy=0 0 3.141592653589793 -> xyz=0.7951 0 0 rpy=0 0 3.141592653589793

File: urdf/dual_gp4.urdf (robot description, URDF)
Before this commit: robot dual_gp4, 30 links, 29 joints
Joints:
- joint left_arm_to_base: origin xyz=-0.6 0 1 rpy=0 0 0 -> xyz=0 0 0 rpy=0 0 0
- joint right_arm_to_base: origin xyz=0.6 0 1 rpy=0 0 3.141592653589793 -> xyz=0.7951 0 0 rpy=0 0 3.141592653589793

File: urdf/dual_gp4.xacro (robot description, xacro)
@@ -10,5 +10,5 @@
     <link name="base">
         <visual>
-            <origin xyz="0 0 0.5" rpy="0 0 0" />
+            <origin xyz="0 0 -0.5" rpy="0 0 0" />
             <geometry>z
                 <box size="2 2 1" />
@@ -19,5 +19,5 @@
         </visual>
         <collision>
-            <origin xyz="0 0 0.5" rpy="0 0 0" />
+            <origin xyz="0 0 -0.5" rpy="0 0 0" />
             <geometry>
                 <box size="2 2 1" />
@@ -35,11 +35,11 @@
         <origin xyz="0.0 0.0 0.0" rpy="0.0 0.0 0.0"/>
     </joint>
+    <!-- left arm -->
+    <xacro:Yaskawa_gp4 arm_id="$(arg arm_id_1)" connected_to="base" xyz="0 0 0" rpy="0 0 0" />
+    <!-- left arm gazebo -->
+    <xacro:gp4_gazebo arm_id="$(arg arm_id_1)" />
     <!-- right arm -->
-    <xacro:Yaskawa_gp4 arm_id="$(arg arm_id_1)" connected_to="base" xyz="-0.6 0 1" rpy="0 0 0" />
-    <!-- right arm gazebo -->
-    <xacro:gp4_gazebo arm_id="$(arg arm_id_1)" />
-    <!-- left arm -->
-    <xacro:Yaskawa_gp4 arm_id="$(arg arm_id_2)" connected_to="base" xyz="0.6 0 1" rpy="0 0 ${pi}" />
-    <!-- left arm gazebo-->
+    <xacro:Yaskawa_gp4 arm_id="$(arg arm_id_2)" connected_to="base" xyz="0.7951 0 0" rpy="0 0 ${pi}" />
+    <!-- right arm gazebo-->
     <xacro:gp4_gazebo arm_id="$(arg arm_id_2)" />
     <!-- load ros_control plugin -->
