Commit message: update gen3 mesh

File: gazebo/urdf/gp4.xacro (robot description, xacro)
@@ -324,5 +324,5 @@
         <origin xyz="0 0 0" rpy="0 0 0"/>
         <geometry>
-          <mesh filename="file://$(find robot_digital_twin)/meshes/eoat/tool_with_cam.stl"/>
+          <mesh filename="file://$(find robot_digital_twin)/meshes/eoat/tool_with_cam_gen35.stl"/>
         </geometry>
         <xacro:material_yaskawa_silver />

File: gazebo/urdf/single_gp4.xacro (robot description, xacro)
@@ -330,5 +330,5 @@
       <origin xyz="0 0 0" rpy="0 0 0"/>
       <geometry>
-        <mesh filename="file://$(find robot_digital_twin)/meshes/eoat/tool_with_cam.stl"/>
+        <mesh filename="file://$(find robot_digital_twin)/meshes/eoat/tool_with_cam_gen35.stl"/>
       </geometry>
     </collision>
@@ -336,5 +336,5 @@
         <origin xyz="0 0 0" rpy="0 0 0"/>
         <geometry>
-          <mesh filename="file://$(find robot_digital_twin)/meshes/eoat/tool_with_cam.stl"/>
+          <mesh filename="file://$(find robot_digital_twin)/meshes/eoat/tool_with_cam_gen35.stl"/>
         </geometry>
         <xacro:material_yaskawa_silver />

File: moveit_config/config/gazebo_dual_gp4.urdf (robot description, URDF)
Before this commit: robot dual_gp4, 32 links, 31 joints
Links:
- removed link left_arm_link_camera
- removed link left_arm_link_camera_origin
- removed link left_arm_link_mountplate
- removed link left_arm_link_precam
- removed link right_arm_link_camera
- removed link right_arm_link_camera_origin
- removed link right_arm_link_mountplate
- removed link right_arm_link_precam
- link left_arm_base_link: geometry collision mesh filename=file:///home/mfi/repos/ros1_ws/src/ruixuan/Robot_Digital_Tw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; visual mesh filename=file:///home/mfi/repos/ros1_ws/src/ruixuan/Robot_Digital_Tw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
- link left_arm_link_1: geometry collision mesh filename=file:///home/mfi/repos/ros1_ws/src/ruixuan/Robot_Digital_Tw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; visual mesh filename=file:///home/mfi/repos/ros1_ws/src/ruixuan/Robot_Digital_Tw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
- link left_arm_link_2: geometry collision mesh filename=file:///home/mfi/repos/ros1_ws/src/ruixuan/Robot_Digital_Tw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; visual mesh filename=file:///home/mfi/repos/ros1_ws/src/ruixuan/Robot_Digital_Tw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
- link left_arm_link_3: geometry collision mesh filename=file:///home/mfi/repos/ros1_ws/src/ruixuan/Robot_Digital_Tw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; visual mesh filename=file:///home/mfi/repos/ros1_ws/src/ruixuan/Robot_Digital_Tw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
- link left_arm_link_4: geometry collision mesh filename=file:///home/mfi/repos/ros1_ws/src/ruixuan/Robot_Digital_Tw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; visual mesh filename=file:///home/mfi/repos/ros1_ws/src/ruixuan/Robot_Digital_Tw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
- link left_arm_link_5: geometry collision mesh filename=file:///home/mfi/repos/ros1_ws/src/ruixuan/Robot_Digital_Tw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; visual mesh filename=file:///home/mfi/repos/ros1_ws/src/ruixuan/Robot_Digital_Tw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
- link left_arm_link_6: geometry collision mesh filename=file:///home/mfi/repos/ros1_ws/src/ruixuan/Robot_Digital_Tw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; visual mesh filename=file:///home/mfi/repos/ros1_ws/src/ruixuan/Robot_Digital_Tw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
- link left_arm_link_tool: geometry collision mesh filename=file:///home/mfi/repos/ros1_ws/src/ruixuan/Robot_Digital_Tw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; visual mesh filename=file:///home/mfi/repos/ros1_ws/src/ruixuan/Robot_Digital_Tw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
- link right_arm_base_link: geometry collision mesh filename=file:///home/mfi/repos/ros1_ws/src/ruixuan/Robot_Digital_Tw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; visual mesh filename=file:///home/mfi/repos/ros1_ws/src/ruixuan/Robot_Digital_Tw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
- link right_arm_link_1: geometry collision mesh filename=file:///home/mfi/repos/ros1_ws/src/ruixuan/Robot_Digital_Tw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; visual mesh filename=file:///home/mfi/repos/ros1_ws/src/ruixuan/Robot_Digital_Tw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
- link right_arm_link_2: geometry collision mesh filename=file:///home/mfi/repos/ros1_ws/src/ruixuan/Robot_Digital_Tw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; visual mesh filename=file:///home/mfi/repos/ros1_ws/src/ruixuan/Robot_Digital_Tw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
- link right_arm_link_3: geometry collision mesh filename=file:///home/mfi/repos/ros1_ws/src/ruixuan/Robot_Digital_Tw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; visual mesh filename=file:///home/mfi/repos/ros1_ws/src/ruixuan/Robot_Digital_Tw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
- link right_arm_link_4: geometry collision mesh filename=file:///home/mfi/repos/ros1_ws/src/ruixuan/Robot_Digital_Tw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; visual mesh filename=file:///home/mfi/repos/ros1_ws/src/ruixuan/Robot_Digital_Tw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
- link right_arm_link_5: geometry collision mesh filename=file:///home/mfi/repos/ros1_ws/src/ruixuan/Robot_Digital_Tw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; visual mesh filename=file:///home/mfi/repos/ros1_ws/src/ruixuan/Robot_Digital_Tw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
- link right_arm_link_6: geometry collision mesh filename=file:///home/mfi/repos/ros1_ws/src/ruixuan/Robot_Digital_Tw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; visual mesh filename=file:///home/mfi/repos/ros1_ws/src/ruixuan/Robot_Digital_Tw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
- link right_arm_link_tool: geometry collision mesh filename=file:///home/mfi/repos/ros1_ws/src/ruixuan/Robot_Digital_Tw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; visual mesh filename=file:///home/mfi/repos/ros1_ws/src/ruixuan/Robot_Digital_Tw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
Joints:
- removed joint left_arm_camera_imgplane
- removed joint left_arm_fts_plate
- removed joint left_arm_plate_precam
- removed joint left_arm_precam_camera
- removed joint right_arm_camera_imgplane
- removed joint right_arm_fts_plate
- removed joint right_arm_plate_precam
- removed joint right_arm_precam_camera
- joint left_arm_fts_tool: origin xyz=0 0 0.027790000000000002 rpy=0 0 3.141592653589793 -> xyz=0 0 0.02525 rpy=0 0 3.141592653589793
- joint left_arm_joint_1: limit (none) -> lower=-2.9670597283903604 upper=2.9670597283903604 effort=0 velocity=8.115781021773632; type continuous -> revolute
- joint left_arm_joint_2: limit (none) -> lower=-1.9198621771937625 upper=2.2689280275926285 effort=100 velocity=8.115781021773632; type continuous -> revolute
- joint left_arm_joint_3: limit (none) -> lower=-1.1344640137963142 upper=3.490658503988659 effort=0 velocity=9.16297857297023; type continuous -> revolute
- joint left_arm_joint_4: limit (none) -> lower=-3.490658503988659 upper=3.490658503988659 effort=0 velocity=9.599310885968812; type continuous -> revolute
- joint left_arm_joint_5: limit (none) -> lower=-2.1467549799530254 upper=2.1467549799530254 effort=0 velocity=9.512044423369096; type continuous -> revolute
- joint left_arm_joint_6: limit (none) -> lower=-7.941248096574199 upper=7.941248096574199 effort=0 velocity=17.453292519943297; type continuous -> revolute
- joint right_arm_fts_tool: origin xyz=0 0 0.027790000000000002 rpy=0 0 3.141592653589793 -> xyz=0 0 0.02525 rpy=0 0 3.141592653589793
- joint right_arm_joint_1: limit (none) -> lower=-2.9670597283903604 upper=2.9670597283903604 effort=0 velocity=8.115781021773632; type continuous -> revolute
- joint right_arm_joint_2: limit (none) -> lower=-1.9198621771937625 upper=2.2689280275926285 effort=100 velocity=8.115781021773632; type continuous -> revolute
- joint right_arm_joint_3: limit (none) -> lower=-1.1344640137963142 upper=3.490658503988659 effort=0 velocity=9.16297857297023; type continuous -> revolute
- joint right_arm_joint_4: limit (none) -> lower=-3.490658503988659 upper=3.490658503988659 effort=0 velocity=9.599310885968812; type continuous -> revolute
- joint right_arm_joint_5: limit (none) -> lower=-2.1467549799530254 upper=2.1467549799530254 effort=0 velocity=9.512044423369096; type continuous -> revolute
- joint right_arm_joint_6: limit (none) -> lower=-7.941248096574199 upper=7.941248096574199 effort=0 velocity=17.453292519943297; type continuous -> revolute
- joint right_arm_to_base: origin xyz=0.88047659 -0.01305078 0.9246 rpy=0 0 3.13422265 -> xyz=0.88101137 -0.01304334 0.92460000 rpy=0 0 3.13585279
