Commit message: revert to gen2 tool in gen2 branch

File: gazebo/urdf/single_gp4.xacro (robot description, xacro)
@@ -330,5 +330,5 @@
       <origin xyz="0 0 0" rpy="0 0 0"/>
       <geometry>
-        <mesh filename="file://$(find robot_digital_twin)/meshes/eoat/tool_with_cam_gen35.stl"/>
+        <mesh filename="file://$(find robot_digital_twin)/meshes/eoat/tool.stl"/>
       </geometry>
     </collision>
@@ -336,5 +336,5 @@
         <origin xyz="0 0 0" rpy="0 0 0"/>
         <geometry>
-          <mesh filename="file://$(find robot_digital_twin)/meshes/eoat/tool_with_cam_gen35.stl"/>
+          <mesh filename="file://$(find robot_digital_twin)/meshes/eoat/tool.stl"/>
         </geometry>
         <xacro:material_yaskawa_silver />
