Commit message: update urdf/xacro to be vamp compatiable

File: gazebo/urdf/quad_gp4.urdf.xacro (robot description, xacro)
@@ -5,6 +5,4 @@
     <xacro:arg name="arm_id_2" default="right_arm" />
     <!-- load arm/hand models and utils (which adds the robot inertia tags to be Gazebo-simulation ready) -->
-    <!-- <xacro:include filename="$(find robot_digital_twin)/urdf/single_gp4.xacro" /> -->
-    <!-- using spherized version for consistent vamp-based collision checking -->
     <xacro:include filename="$(find robot_digital_twin)/urdf/single_gp4_spherized.xacro" />
     <link name="world"/>
@@ -19,6 +17,9 @@
     <!-- left arm -->
     <xacro:Yaskawa_gp4 arm_id="$(arg arm_id_1)" connected_to="base" xyz="0 0 0.9246" rpy="0 0 0" />
+    <!-- left arm gazebo -->
     <!-- right arm -->
     <xacro:Yaskawa_gp4 arm_id="$(arg arm_id_2)" connected_to="base" xyz="0.88128092 -0.01226491 0.92460000" rpy="0 0 3.13792336" />
+    <!-- right arm gazebo-->
+    <xacro:gp4_gazebo arm_id="$(arg arm_id_2)" />
     <!-- load ros_control plugin -->
     <gazebo>

File: gazebo/urdf/single_gp4.xacro (robot description, xacro)
@@ -362,5 +362,5 @@
       <origin xyz="0 0 0.260" rpy="0 0 0" />
       <axis xyz="0 -1 0" />
-      <limit effort="0" lower="${radians(-65)}" upper="${radians(200)}" velocity="${radians(525)}" />
+      <limit effort="0" lower="${radians(-56)}" upper="${radians(180)}" velocity="${radians(525)}" />
     </joint>
     <joint name="${arm_id}_joint_4" type="revolute">
@@ -376,5 +376,5 @@
       <origin xyz="0 0 0" rpy="0 0 0" />
       <axis xyz="0 -1 0" />
-      <limit effort="0" lower="${radians(-123)}" upper="${radians(123)}" velocity="${radians(545)}" />
+      <limit effort="0" lower="${radians(-105)}" upper="${radians(105)}" velocity="${radians(545)}" />
     </joint>
     <joint name="${arm_id}_joint_6" type="revolute">
