Commit message: add cam

File: gazebo/urdf/galaxea.xacro (robot description, xacro)
@@ -972,5 +972,5 @@
         rpy="0 0 0" />
       <mass
-        value="0.604" />
+        value="0.05" />
       <inertia
         ixx="0.000175881544189539"
@@ -995,5 +995,5 @@
       </material>
     </visual>
-    <collision>
+    <!-- <collision>
       <origin
         xyz="0 0 0"
@@ -1003,5 +1003,5 @@
           filename="file://$(find robot_digital_twin)/meshes/eoat/galaxea_eoat.STL" />
       </geometry>
-    </collision>
+    </collision> -->
   </link>
   <joint name="left_eoat_joint" type="fixed">
@@ -1009,5 +1009,5 @@
     <parent link="left_arm_link6" />
     <child link="left_arm_eoat" />
-    <axis xyz="0 0 1" />
+    <axis xyz="0 0 0" />
   </joint>
   <link
@@ -1419,5 +1419,5 @@
         rpy="0 0 0" />
       <mass
-        value="0.604" />
+        value="0.05" />
       <inertia
         ixx="0.000175881544189539"
@@ -1442,5 +1442,5 @@
       </material>
     </visual>
-    <collision>
+    <!-- <collision>
       <origin
         xyz="0 0 0"
@@ -1450,5 +1450,5 @@
           filename="file://$(find robot_digital_twin)/meshes/eoat/galaxea_eoat.STL" />
       </geometry>
-    </collision>
+    </collision> -->
   </link>
   <joint name="right_eoat_joint" type="fixed">
@@ -1456,5 +1456,5 @@
     <parent link="right_arm_link6" />
     <child link="right_arm_eoat" />
-    <axis xyz="0 0 1" />
+    <axis xyz="0 0 0" />
   </joint>
   </xacro:macro>
@@ -1501,4 +1501,42 @@
     </plugin>
   </gazebo>
+  <xacro:include filename="$(find realsense_gazebo_description)/urdf/_d435i.urdf.xacro"/>
+  <xacro:sensor_d435i parent="torso_link3"
+                      name="head_camera"
+                      topics_ns="/galaxea/head_camera"
+                      color_width="1280"
+                      color_height="720"
+                      color_fps="15"
+                      enable_pointCloud="true"
+                      depth_width="1280"
+                      depth_height="720"
+                      depth_fps="15" >
+      <origin xyz="0 0 0.4" rpy="0 ${pi/4} 0"/>
+  </xacro:sensor_d435i>
+  <xacro:include filename="$(find realsense_gazebo_description)/urdf/_d405.urdf.xacro"/>
+  <xacro:sensor_d405 parent="left_arm_eoat"
+                        name="left_wrist_camera"
+                        topics_ns="/galaxea/left_wrist_camera"
+                        color_width="1280"
+                        color_height="720"
+                        color_fps="15"
+                        enable_pointCloud="true"
+                        depth_width="1280"
+                        depth_height="720"
+                        depth_fps="15" >
+      <origin xyz="-0.095 0 0.08" rpy="0 ${pi/4} 0"/>
+  </xacro:sensor_d405>
+  <xacro:sensor_d405 parent="right_arm_eoat"
+                        name="right_wrist_camera"
+                        topics_ns="/galaxea/right_wrist_camera"
+                        color_width="1280"
+                        color_height="720"
+                        color_fps="15"
+                        enable_pointCloud="true"
+                        depth_width="1280"
+                        depth_height="720"
+                        depth_fps="15" >
+      <origin xyz="-0.095 0 0.08" rpy="0 ${pi/4} 0"/>
+  </xacro:sensor_d405>
   <gazebo reference="base">
     <material>Galaxea/Grey</material>

Commit message: add virtual links

File: gazebo/urdf/galaxea.xacro (robot description, xacro)
@@ -1011,4 +1011,34 @@
     <axis xyz="0 0 0" />
   </joint>
+  <link name = "left_tmp1"/>
+  <joint name = "left_tool_tmp1_joint" type="fixed">
+    <parent link = "left_arm_eoat" />
+    <child link = "left_tmp1" />
+    <origin xyz="0 0 0" rpy="-${pi/4} 0 0" />
+  </joint>
+  <link name = "left_tmp2"/>
+  <joint name = "left_tmp1_tmp2_joint" type="fixed">
+    <parent link = "left_tmp1" />
+    <child link = "left_tmp2" />
+    <origin xyz="0 0 0" rpy="0 -${pi/2} 0" />
+  </joint>
+  <link name = "left_attach"/>
+  <joint name = "left_tmp2_attach_joint" type="fixed">
+    <parent link = "left_tmp2" />
+    <child link = "left_attach" />
+    <origin xyz="0 0 0.0032" rpy="0 0 0" />
+  </joint>
+  <link name = "left_assemble"/>
+  <joint name = "left_attach_assemble_joint" type="fixed">
+    <parent link = "left_attach" />
+    <child link = "left_assemble" />
+    <origin xyz="0.008 0 0" rpy="0 0 0" />
+  </joint>
+  <link name = "left_disassemble"/>
+  <joint name = "left_attach_disassemble_joint" type="fixed">
+    <parent link = "left_attach" />
+    <child link = "left_disassemble" />
+    <origin xyz="0 0 -0.0096" rpy="0 0 0" />
+  </joint>
   <link
     name="right_arm_base_link">
@@ -1457,4 +1487,34 @@
     <child link="right_arm_eoat" />
     <axis xyz="0 0 0" />
+  </joint>
+  <link name = "right_tmp1"/>
+  <joint name = "right_tool_tmp1_joint" type="fixed">
+    <parent link = "right_arm_eoat" />
+    <child link = "right_tmp1" />
+    <origin xyz="0 0 0" rpy="-${pi/4} 0 0" />
+  </joint>
+  <link name = "right_tmp2"/>
+  <joint name = "right_tmp1_tmp2_joint" type="fixed">
+    <parent link = "right_tmp1" />
+    <child link = "right_tmp2" />
+    <origin xyz="0 0 0" rpy="0 -${pi/2} 0" />
+  </joint>
+  <link name = "right_attach"/>
+  <joint name = "right_tmp2_attach_joint" type="fixed">
+    <parent link = "right_tmp2" />
+    <child link = "right_attach" />
+    <origin xyz="0 0 0.0032" rpy="0 0 0" />
+  </joint>
+  <link name = "right_assemble"/>
+  <joint name = "right_attach_assemble_joint" type="fixed">
+    <parent link = "right_attach" />
+    <child link = "right_assemble" />
+    <origin xyz="0.008 0 0" rpy="0 0 0" />
+  </joint>
+  <link name = "right_disassemble"/>
+  <joint name = "right_attach_disassemble_joint" type="fixed">
+    <parent link = "right_attach" />
+    <child link = "right_disassemble" />
+    <origin xyz="0 0 -0.0096" rpy="0 0 0" />
   </joint>
   </xacro:macro>
