Commit message: update urdf

File: gazebo/urdf/galaxea.urdf (robot description, URDF)
Before this commit: robot galaxea_r1_lite, 62 links, 61 joints
Links:
- added link left_assemble
- added link left_attach
- added link left_disassemble
- added link left_tmp1
- added link left_tmp2
- added link right_assemble
- added link right_attach
- added link right_disassemble
- added link right_tmp1
- added link right_tmp2
Joints:
- added joint left_attach_assemble_joint: type fixed, parent left_attach, child left_assemble, origin xyz=0.008 0 0 rpy=0 0 0
- added joint left_attach_disassemble_joint: type fixed, parent left_attach, child left_disassemble, origin xyz=0 0 -0.0096 rpy=0 0 0
- added joint left_tmp1_tmp2_joint: type fixed, parent left_tmp1, child left_tmp2, origin xyz=0 0 0 rpy=0 -1.5707963267948966 0
- added joint left_tmp2_attach_joint: type fixed, parent left_tmp2, child left_attach, origin xyz=0 0 0.0032 rpy=0 0 0
- added joint left_tool_tmp1_joint: type fixed, parent left_arm_eoat, child left_tmp1, origin xyz=0 0 0 rpy=-0.7853981633974483 0 0
- added joint right_attach_assemble_joint: type fixed, parent right_attach, child right_assemble, origin xyz=0.008 0 0 rpy=0 0 0
- added joint right_attach_disassemble_joint: type fixed, parent right_attach, child right_disassemble, origin xyz=0 0 -0.0096 rpy=0 0 0
- added joint right_tmp1_tmp2_joint: type fixed, parent right_tmp1, child right_tmp2, origin xyz=0 0 0 rpy=0 -1.5707963267948966 0
- added joint right_tmp2_attach_joint: type fixed, parent right_tmp2, child right_attach, origin xyz=0 0 0.0032 rpy=0 0 0
- added joint right_tool_tmp1_joint: type fixed, parent right_arm_eoat, child right_tmp1, origin xyz=0 0 0 rpy=-0.7853981633974483 0 0
